File: SGX-CH4-sensor/SGX-CH4-sensor/SGX-CH4-sensor.sch (KiCad schematic (older format))
At the start: 3 parts

Commit message: fewf
Parts:
- removed D? (x2): D_Zener, symbol Device:D_Zener
- added C1: C, Capacitor_THT:CP_Radial_D8.0mm_P5.00mm, symbol Device:C
- added C2: 10n, Capacitor_THT:CP_Radial_D6.3mm_P2.50mm, symbol Device:C
- added D1, D2: D_Zener, Diode_THT:D_DO-35_SOD27_P10.16mm_Horizontal, symbol Device:D_Zener
- added F1: Fuse, Resistor_THT:R_Axial_DIN0309_L9.0mm_D3.2mm_P5.08mm_Vertical, symbol Device:Fuse
- added J1: Conn_01x05_Male, Connector_PinHeader_2.54mm:PinHeader_1x05_P2.54mm_Vertical, symbol Connector:Conn_01x05_Male
- added J2, J8, J9: tx, Connector_PinHeader_2.54mm:PinHeader_1x01_P2.54mm_Vertical, symbol Connector:Conn_01x01_Male
- added J3: rx, Connector_PinHeader_2.54mm:PinHeader_1x01_P2.54mm_Vertical, symbol Connector:Conn_01x01_Male
- added J4: analog out, Connector_PinHeader_2.54mm:PinHeader_1x01_P2.54mm_Vertical, symbol Connector:Conn_01x01_Male
- added J5: gnd, Connector_PinHeader_2.54mm:PinHeader_1x01_P2.54mm_Vertical, symbol Connector:Conn_01x01_Male
- added J6: v in, Connector_PinHeader_2.54mm:PinHeader_1x01_P2.54mm_Vertical, symbol Connector:Conn_01x01_Male
- added TP1, TP2, TP3, TP4, TP5, TP6: TestPoint, TestPoint:TestPoint_Pad_D3.0mm, symbol Connector:TestPoint
- added U1: AD8603, Package_TO_SOT_SMD:SOT-23-5, symbol Amplifier_Operational:AD8603
- D3: renamed from D?; footprint (none) -> Diode_THT:D_DO-35_SOD27_P10.16mm_Horizontal
Connections:
- net at D3.1 (K): now also C1.1, C2.1, D1.1 (K), D2.1 (K), J1.2 (Pin_2), J1.3 (Pin_3), J6.1 (Pin_1), TP1.1, U1.5 (V+)
- net at D3.2 (A): now also C2.2, D1.2 (A), D2.2 (A), F1.1, J5.1 (Pin_1), TP2.1, TP4.1, U1.2 (V-)
- new net: J2.1 (Pin_1), J8.1 (Pin_1), TP5.1
- new net: J3.1 (Pin_1), J9.1 (Pin_1), TP6.1
- new net: J4.1 (Pin_1), U1.3 (+)
- new net: J1.1 (Pin_1), TP3.1, U1.1, U1.4 (-)
- new net GND: C1.2, F1.2, J1.4 (Pin_4), J1.5 (Pin_5)

Commit message: hthet
Parts:
- removed J1: Conn_01x05_Male, Connector_PinHeader_2.54mm:PinHeader_1x05_P2.54mm_Vertical, symbol Connector:Conn_01x05_Male
- added J1: Conn_01x03_Male, Connector_PinHeader_2.54mm:PinHeader_1x03_P2.54mm_Vertical, symbol Connector:Conn_01x03_Male
- J8: value tx -> tx2
- J9: value tx -> rx2
Connections:
- net GND: now also J1.3 (Pin_3)
- net at C1.1, C2.1, D1.1 (K)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: now also J1.2 (Pin_2)
- net at TP3.1, U1.1, U1.4 (-): now also J1.1 (Pin_1)
Other:
- moved on the sheet: J3, J9, TP6
Changed lines of the file:
@@
 L Connector:Conn_01x01_Male J3
 U 1 1 60ACC117
-P 5450 2600
-F 0 "J3" H 5422 2532 50  0000 R CNN
-F 1 "rx" H 5422 2623 50  0000 R CNN
-F 2 "Connector_PinHeader_2.54mm:PinHeader_1x01_P2.54mm_Vertical" H 5450 2600 50  0001 C CNN
-F 3 "~" H 5450 2600 50  0001 C CNN
-	1    5450 2600
+P 5650 2900
+F 0 "J3" H 5622 2832 50  0000 R CNN
+F 1 "rx" H 5622 2923 50  0000 R CNN
+F 2 "Connector_PinHeader_2.54mm:PinHeader_1x01_P2.54mm_Vertical" H 5650 2900 50  0001 C CNN
+F 3 "~" H 5650 2900 50  0001 C CNN
+	1    5650 2900
 	-1   0    0    1
 $EndComp
@@
 $EndComp
 $Comp
-L Connector:Conn_01x05_Male J1
-U 1 1 60ACE4A7
-P 1000 2550
-F 0 "J1" H 1108 2931 50  0000 C CNN
-F 1 "Conn_01x05_Male" H 1108 2840 50  0000 C CNN
-F 2 "Connector_PinHeader_2.54mm:PinHeader_1x05_P2.54mm_Vertical" H 1000 2550 50  0001 C CNN
-F 3 "~" H 1000 2550 50  0001 C CNN
-	1    1000 2550
-	1    0    0    -1
-$EndComp
-$Comp
 L Amplifier_Operational:AD8603 U1
 U 1 1 60ACF53E
@@
 $EndComp
 Wire Wire Line
-	1200 2650 1200 2750
-Wire Wire Line
 	1200 3150 1650 3150
 Wire Wire Line
@@
 Wire Wire Line
 	2550 3150 2700 3150
-Connection ~ 1200 2750
-Wire Wire Line
-	1200 2750 1200 3150
 Connection ~ 1650 3150
 Wire Wire Line
@@
 Wire Wire Line
 	1950 2700 1300 2700
-Wire Wire Line
-	1300 2450 1200 2450
-Wire Wire Line
-	1200 2550 1200 2450
-Connection ~ 1200 2450
 Connection ~ 3350 3000
 Wire Wire Line
@@
 P 4950 2500
 F 0 "J8" H 5058 2681 50  0000 C CNN
-F 1 "tx" H 5058 2590 50  0000 C CNN
+F 1 "tx2" H 5058 2590 50  0000 C CNN
 F 2 "Connector_PinHeader_2.54mm:PinHeader_1x01_P2.54mm_Vertical" H 4950 2500 50  0001 C CNN
 F 3 "~" H 4950 2500 50  0001 C CNN
@@
 L Connector:Conn_01x01_Male J9
 U 1 1 60AE0110
-P 4950 2600
-F 0 "J9" H 5058 2781 50  0000 C CNN
-F 1 "tx" H 5058 2690 50  0000 C CNN
-F 2 "Connector_PinHeader_2.54mm:PinHeader_1x01_P2.54mm_Vertical" H 4950 2600 50  0001 C CNN
-F 3 "~" H 4950 2600 50  0001 C CNN
-	1    4950 2600
+P 5150 2900
+F 0 "J9" H 5258 3081 50  0000 C CNN
+F 1 "rx2" H 5258 2990 50  0000 C CNN
+F 2 "Connector_PinHeader_2.54mm:PinHeader_1x01_P2.54mm_Vertical" H 5150 2900 50  0001 C CNN
+F 3 "~" H 5150 2900 50  0001 C CNN
+	1    5150 2900
 	1    0    0    -1
 $EndComp
@@
 	5150 2500 5200 2500
 Wire Wire Line
-	5250 2600 5200 2600
+	5450 2900 5400 2900
 Wire Wire Line
 	1950 2700 2400 2700
@@
 L Connector:TestPoint TP6
 U 1 1 60AE5045
-P 5200 2600
-F 0 "TP6" H 5142 2626 50  0000 R CNN
-F 1 "TestPoint" H 5142 2717 50  0000 R CNN
-F 2 "TestPoint:TestPoint_Pad_D3.0mm" H 5400 2600 50  0001 C CNN
-F 3 "~" H 5400 2600 50  0001 C CNN
-	1    5200 2600
-	-1   0    0    1
-$EndComp
-Connection ~ 5200 2600
-Wire Wire Line
-	5200 2600 5150 2600
+P 5400 2900
+F 0 "TP6" H 5342 2926 50  0000 R CNN
+F 1 "TestPoint" H 5342 3017 50  0000 R CNN
+F 2 "TestPoint:TestPoint_Pad_D3.0mm" H 5600 2900 50  0001 C CNN
+F 3 "~" H 5600 2900 50  0001 C CNN
+	1    5400 2900
+	-1   0    0    1
+$EndComp
+Connection ~ 5400 2900
+Wire Wire Line
+	5400 2900 5350 2900
 Wire Wire Line
 	4350 2300 4350 2800
@@
 Wire Wire Line
 	3750 2600 3750 2400
+$Comp
+L Connector:Conn_01x03_Male J1
+U 1 1 60B03AF6
+P 1000 2450
+F 0 "J1" H 1108 2731 50  0000 C CNN
+F 1 "Conn_01x03_Male" H 1108 2640 50  0000 C CNN
+F 2 "Connector_PinHeader_2.54mm:PinHeader_1x03_P2.54mm_Vertical" H 1000 2450 50  0001 C CNN
+F 3 "~" H 1000 2450 50  0001 C CNN
+	1    1000 2450
+	1    0    0    -1
+$EndComp
+Wire Wire Line
+	1200 2550 1200 3150
+Wire Wire Line
+	1200 2450 1300 2450
 $EndSCHEMATC
