File: SGX-CH4-sensor/SGX-CH4-sensor/SGX-CH4-sensor.kicad_pcb (KiCad board)
At the start: 2 copper layers, 22 parts, among them J1 Conn_01x05_Male, J2 tx, J3 rx, J4 analog out, J5 gnd, J6 v in, J7 tx, J8 tx, J9 tx, U1 AD8603

Commit message: hthet
Parts:
- removed J7: tx, Connector_PinHeader_2.54mm:PinHeader_1x01_P2.54mm_Vertical
- J1: value Conn_01x05_Male -> Conn_01x03_Male; footprint Connector_PinHeader_2.54mm:PinHeader_1x05_P2.54mm_Vertical -> Connector_PinHeader_2.54mm:PinHeader_1x03_P2.54mm_Vertical
- J8: value tx -> tx2
- J9: value tx -> rx2
- TP1, TP4, TP5, TP6: moved to B.Cu
- moved J5 92.5 mm to (132.7, 116.2), turned to 180 degrees
- moved J2 91.0 mm to (125.7, 98.4), turned to 180 degrees
- moved J6 91.0 mm to (137.2, 106.7), turned to 180 degrees
- moved J3 87.8 mm to (117.5, 116.2), turned to 180 degrees
- moved J9 78.3 mm to (111.8, 116.2), turned to 180 degrees
- moved J4 78.1 mm to (115.6, 106.0), turned to 180 degrees
- moved F1 76.3 mm to (78.7, 110.5), turned to 180 degrees
- moved J8 76.1 mm to (132.7, 98.4), turned to 180 degrees
- moved U1 76.1 mm to (108.1, 105.1)
- moved TP5 75.1 mm to (121.3, 98.4), turned to 180 degrees
- moved D2 73.5 mm to (85.1, 100.3), turned to 270 degrees
- moved C2 71.8 mm to (101.0, 104.1), turned to 270 degrees
- moved J1 69.5 mm to (63.2, 102.9)
- moved TP6 69.0 mm to (107.3, 116.2), turned to 180 degrees
- moved D1 68.1 mm to (93.1, 100.1), turned to 270 degrees
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Connections:
- J1 pad 3: Net-(C1-Pad1) -> GND
Routing:
- net Net-(C1-Pad1): track 0.00 -> 93.5 mm, vias 0 -> 1
- net Net-(C2-Pad2): track 0.00 -> 77.3 mm
- net Net-(J1-Pad1): track 0.00 -> 69.8 mm, vias 0 -> 2
- net GND: track 0.00 -> 18.0 mm
- net Net-(J4-Pad1): track 0.00 -> 12.5 mm
- net Net-(J2-Pad1): track 0.00 -> 11.4 mm
- net Net-(J3-Pad1): track 0.00 -> 10.2 mm
- net (no net): track 0.00 -> 10.0 mm
Other:
- board outline added: 80 x 30 mm
- board text added: "1 CM"

Commit message: fewfew
Parts:
- moved TP5 3.42 mm to (120.0, 95.2)
Routing:
- net Net-(J1-Pad1): track 69.8 -> 111.1 mm
- net Net-(C1-Pad1): track 93.5 -> 124.7 mm
- net Net-(C2-Pad2): track 77.3 -> 81.1 mm
- net Net-(J2-Pad1): track 11.4 -> 14.0 mm
