File: irigatii/irigatii.sch (KiCad schematic (older format))
At the start: 29 parts

Commit message: 4t
Parts:
- removed M?: MNMOS, symbol pspice:MNMOS
- removed R? (x2): R, symbol Device:R
- added D? (x2): D, symbol Device:D
- added M? (x2): Motor_DC, symbol Motor:Motor_DC
- added Q?: Q_NMOS_GSD, symbol Device:Q_NMOS_GSD
Connections:
- net 0: now also Q?.3 (D)
- net pincontrol: now also Q?.1 (G)
- net at K?.4: now also D?.1 (K), M?.1 (+) (x2)
- net at K?.7: now also D?.2 (A), M?.2 (-) (x2)
- net at D?.1 (K), K?.1: now also Q?.2 (S)
Other:
- moved on the sheet: D?, K?
Changed lines of the file:
@@
 Wire Wire Line
 	3200 1350 3400 1350
-$Comp
-L Device:R R?
-U 1 1 60D1F8D5
-P 4500 1900
-F 0 "R?" H 4570 1946 50  0000 L CNN
-F 1 "R" H 4570 1855 50  0000 L CNN
-F 2 "" V 4430 1900 50  0001 C CNN
-F 3 "~" H 4500 1900 50  0001 C CNN
-	1    4500 1900
-	1    0    0    -1
-$EndComp
 Text Label 1700 1700 0    50   ~ 0
 L1
@@
 Wire Wire Line
 	3400 1950 3400 2150
-Wire Wire Line
-	4000 1850 4350 1850
-Wire Wire Line
-	4350 1850 4350 1750
-Wire Wire Line
-	4350 1750 4500 1750
-Wire Wire Line
-	4500 2050 4500 2250
-Wire Wire Line
-	4500 2250 4000 2250
 Wire Wire Line
 	3850 950  4000 950
@@
 L Relay:AZ850-x K?
 U 1 1 60D277D4
-P 7450 1900
-F 0 "K?" V 6683 1900 50  0000 C CNN
-F 1 "AZ850-x" V 6774 1900 50  0000 C CNN
-F 2 "Relay_THT:Relay_DPDT_FRT5" H 8000 1950 50  0001 C CNN
-F 3 "http://www.azettler.com/pdfs/az850.pdf" H 7450 1900 50  0001 C CNN
-	1    7450 1900
+P 3150 4550
+F 0 "K?" V 2383 4550 50  0000 C CNN
+F 1 "AZ850-x" V 2474 4550 50  0000 C CNN
+F 2 "Relay_THT:Relay_DPDT_FRT5" H 3700 4600 50  0001 C CNN
+F 3 "http://www.azettler.com/pdfs/az850.pdf" H 3150 4550 50  0001 C CNN
+	1    3150 4550
 	0    1    1    0
 $EndComp
@@
 L Device:D D?
 U 1 1 60D277DA
-P 7450 1100
-F 0 "D?" H 7450 883 50  0000 C CNN
-F 1 "D" H 7450 974 50  0000 C CNN
-F 2 "" H 7450 1100 50  0001 C CNN
-F 3 "~" H 7450 1100 50  0001 C CNN
-	1    7450 1100
+P 3150 3750
+F 0 "D?" H 3150 3533 50  0000 C CNN
+F 1 "D" H 3150 3624 50  0000 C CNN
+F 2 "" H 3150 3750 50  0001 C CNN
+F 3 "~" H 3150 3750 50  0001 C CNN
+	1    3150 3750
 	-1   0    0    1
 $EndComp
-Text Label 8100 850  0    50   ~ 0
+Text Label 3800 3500 0    50   ~ 0
 pincontrol
 Wire Wire Line
-	7750 950  7750 1100
-Wire Wire Line
-	5900 1500 6950 1500
-Wire Wire Line
-	7300 1100 6950 1100
-Wire Wire Line
-	6950 1100 6950 1500
-Connection ~ 6950 1500
-Wire Wire Line
-	6950 1500 7150 1500
-$Comp
-L Device:R R?
-U 1 1 60D277E7
-P 8250 2050
-F 0 "R?" H 8320 2096 50  0000 L CNN
-F 1 "R" H 8320 2005 50  0000 L CNN
-F 2 "" V 8180 2050 50  0001 C CNN
-F 3 "~" H 8250 2050 50  0001 C CNN
-	1    8250 2050
-	1    0    0    -1
-$EndComp
-Text Label 5450 1850 0    50   ~ 0
+	3450 3600 3450 3750
+Wire Wire Line
+	1600 4150 2650 4150
+Wire Wire Line
+	3000 3750 2650 3750
+Wire Wire Line
+	2650 3750 2650 4150
+Connection ~ 2650 4150
+Wire Wire Line
+	2650 4150 2850 4150
+Text Label 1150 4500 0    50   ~ 0
 L1
-Text Label 5450 2100 0    50   ~ 0
+Text Label 1150 4750 0    50   ~ 0
 L2
 Wire Wire Line
-	5450 1850 7150 1850
-Wire Wire Line
-	7150 1850 7150 1900
-Wire Wire Line
-	5450 2100 7150 2100
-Wire Wire Line
-	7150 2100 7150 2300
-Wire Wire Line
-	7750 2000 8100 2000
-Wire Wire Line
-	8100 2000 8100 1900
-Wire Wire Line
-	8100 1900 8250 1900
-Wire Wire Line
-	8250 2200 8250 2400
-Wire Wire Line
-	8250 2400 7750 2400
-Wire Wire Line
-	7600 1100 7750 1100
-Connection ~ 7750 1100
-Wire Wire Line
-	7750 1100 7750 1500
+	1150 4500 2850 4500
+Wire Wire Line
+	2850 4500 2850 4550
+Wire Wire Line
+	1150 4750 2850 4750
+Wire Wire Line
+	2850 4750 2850 4950
+Wire Wire Line
+	3300 3750 3450 3750
+Connection ~ 3450 3750
+Wire Wire Line
+	3450 3750 3450 4150
 $Comp
 L pspice:0 #GND?
 U 1 1 60D277FB
-P 5900 1500
-F 0 "#GND?" H 5900 1400 50  0001 C CNN
-F 1 "0" H 5900 1589 50  0000 C CNN
-F 2 "" H 5900 1500 50  0001 C CNN
-F 3 "~" H 5900 1500 50  0001 C CNN
-	1    5900 1500
-	1    0    0    -1
-$EndComp
-$Comp
-L pspice:MNMOS M?
-U 1 1 60D2AACE
-P 7850 750
-F 0 "M?" H 8137 796 50  0000 L CNN
-F 1 "MNMOS" H 8137 705 50  0000 L CNN
-F 2 "" H 7825 750 50  0001 C CNN
-F 3 "~" H 7825 750 50  0001 C CNN
-	1    7850 750
-	-1   0    0    -1
-$EndComp
-Wire Wire Line
-	7650 950  7750 950
-Connection ~ 7750 950
-Wire Wire Line
-	8050 750  8050 850
-Wire Wire Line
-	8050 850  8100 850
-Text Label 8100 550  0    50   ~ 0
+P 1600 4150
+F 0 "#GND?" H 1600 4050 50  0001 C CNN
+F 1 "0" H 1600 4239 50  0000 C CNN
+F 2 "" H 1600 4150 50  0001 C CNN
+F 3 "~" H 1600 4150 50  0001 C CNN
+	1    1600 4150
+	1    0    0    -1
+$EndComp
+Wire Wire Line
+	3750 3400 3750 3500
+Wire Wire Line
+	3750 3500 3800 3500
+Text Label 3800 3200 0    50   ~ 0
 +12v
 Wire Wire Line
-	8100 550  7750 550
+	3800 3200 3450 3200
 Text Label 9350 1150 0    50   ~ 0
 +12v
@@
 	14650 4700 14650 2300
 Connection ~ 14650 2300
+$Comp
+L Motor:Motor_DC M?
+U 1 1 60D45F34
+P 4450 2050
+F 0 "M?" H 4608 2046 50  0000 L CNN
+F 1 "Motor_DC" H 4608 1955 50  0000 L CNN
+F 2 "" H 4450 1960 50  0001 C CNN
+F 3 "~" H 4450 1960 50  0001 C CNN
+	1    4450 2050
+	1    0    0    -1
+$EndComp
+$Comp
+L Device:D D?
+U 1 1 60D506D1
+P 4200 2100
+F 0 "D?" H 4200 1883 50  0000 C CNN
+F 1 "D" H 4200 1974 50  0000 C CNN
+F 2 "" H 4200 2100 50  0001 C CNN
+F 3 "~" H 4200 2100 50  0001 C CNN
+	1    4200 2100
+	0    1    1    0
+$EndComp
+Wire Wire Line
+	4000 1850 4200 1850
+Wire Wire Line
+	4450 2350 4000 2350
+Wire Wire Line
+	4000 2350 4000 2250
+Wire Wire Line
+	4000 2250 4200 2250
+Connection ~ 4000 2250
+Wire Wire Line
+	4200 1950 4200 1850
+Connection ~ 4200 1850
+Wire Wire Line
+	4200 1850 4450 1850
+$Comp
+L Motor:Motor_DC M?
+U 1 1 60D629BE
+P 3900 4850
+F 0 "M?" H 4058 4846 50  0000 L CNN
+F 1 "Motor_DC" H 4058 4755 50  0000 L CNN
+F 2 "" H 3900 4760 50  0001 C CNN
+F 3 "~" H 3900 4760 50  0001 C CNN
+	1    3900 4850
+	1    0    0    -1
+$EndComp
+$Comp
+L Device:D D?
+U 1 1 60D629C4
+P 3650 4900
+F 0 "D?" H 3650 4683 50  0000 C CNN
+F 1 "D" H 3650 4774 50  0000 C CNN
+F 2 "" H 3650 4900 50  0001 C CNN
+F 3 "~" H 3650 4900 50  0001 C CNN
+	1    3650 4900
+	0    1    1    0
+$EndComp
+Wire Wire Line
+	3450 4650 3650 4650
+Wire Wire Line
+	3900 5150 3450 5150
+Wire Wire Line
+	3450 5150 3450 5050
+Wire Wire Line
+	3450 5050 3650 5050
+Wire Wire Line
+	3650 4750 3650 4650
+Connection ~ 3650 4650
+Wire Wire Line
+	3650 4650 3900 4650
+Connection ~ 3450 5050
+$Comp
+L Device:Q_NMOS_GSD Q?
+U 1 1 60D701CF
+P 3550 3400
+F 0 "Q?" V 3799 3400 50  0000 C CNN
+F 1 "Q_NMOS_GSD" V 3890 3400 50  0000 C CNN
+F 2 "" H 3750 3500 50  0001 C CNN
+F 3 "~" H 3550 3400 50  0001 C CNN
+	1    3550 3400
+	-1   0    0    -1
+$EndComp
 $EndSCHEMATC
