File: SGX-CH4-sensor_v2/SGX-CH4-sensor_v2.kicad_pcb (KiCad board)
At the start: 2 copper layers, 23 x 63 mm, 9 parts, among them J1 Conn_02x03_Odd_Even, U1 OP179GRT, U2 SGX-INIR-CH4-sensor

Commit message: ef
Routing:
- net Net-(C1-Pad1): track 57.8 -> 76.1 mm, vias 1 -> 3
- net Net-(C1-Pad2): track 51.2 -> 63.0 mm, vias 1 -> 3
- net Net-(J1-Pad6): track 2.28 -> 9.54 mm, vias 1 -> 2
- net Net-(J1-Pad5): track 2.66 -> 7.43 mm, vias 1 -> 2
- net Net-(J1-Pad1): track 5.66 -> 8.44 mm, vias 1 -> 2
