File: 25-station-led-alarm/25-station-led-alarm.kicad_pcb (KiCad board)
At the start: 2 copper layers, 26 parts, among them Q1 Q_NMOS_DGS, Q2 Q_NMOS_DGS, Q3 Q_NMOS_DGS

Commit message: d
Parts:
- added H1: MountingHole_Pad, MountingHole:MountingHole_2.7mm_M2.5, F.Cu at (128.3, 156.1)
- added H2: MountingHole_Pad, MountingHole:MountingHole_2.7mm_M2.5, F.Cu at (127.7, 146.8)
- added H3: MountingHole_Pad, MountingHole:MountingHole_2.7mm_M2.5, F.Cu at (128.4, 91.5)
- added H4: MountingHole_Pad, MountingHole:MountingHole_2.7mm_M2.5, F.Cu at (161.8, 91.2)
- added J1: Conn_02x03_Counter_Clockwise, Connector_PinHeader_2.54mm:PinHeader_2x03_P2.54mm_Horizontal, F.Cu at (141.1, 94.1)
- BZ1: footprint Buzzer_Beeper:Buzzer_TDK_PS1240P02BT_D12.2mm_H6.5mm -> Buzzer_Beeper:resita_buzzer
- D13: value LED_red -> D; footprint LED_THT:LED_D5.0mm -> Diode_THT:D_DO-15_P12.70mm_Horizontal
- moved R9 95.4 mm to (137.8, 143.1), turned to 270 degrees
- moved R8 93.9 mm to (132.8, 153.4), turned to 90 degrees
- moved R7 87.4 mm to (135.0, 116.0), turned to 270 degrees
- moved R5 67.7 mm to (135.0, 111.0), turned to 90 degrees
- moved R1 49.3 mm to (162.0, 143.0), turned to 270 degrees
- moved Q3 45.3 mm to (139.7, 137.6), turned to 180 degrees
- moved R2 45.1 mm to (129.4, 115.8), turned to 90 degrees
- moved Q1 26.9 mm to (142.5, 124.1), turned to 90 degrees
- moved Q2 24.2 mm to (141.5, 112.4), turned to 90 degrees
- moved D13 19.9 mm to (156.5, 157.7), turned to 90 degrees
- moved BZ1 17.8 mm to (146.8, 149.7), turned to 180 degrees
- moved R4 15.5 mm to (129.6, 122.8), turned to 270 degrees
- moved D10 14.5 mm to (153.0, 126.0)
- moved D4 14.2 mm to (160.0, 126.0)
- moved D1 13.9 mm to (160.0, 132.0)
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Routing:
- net /P3: track 0.00 -> 72.5 mm
- net +5V: track 0.00 -> 70.5 mm
- net /P1: track 0.00 -> 47.8 mm
- net Net-(BZ1-Pad2): track 0.00 -> 23.1 mm
- net Net-(D11-Pad1): track 0.00 -> 23.0 mm
- net Net-(Q1-Pad2): track 0.00 -> 18.7 mm
- net Net-(D10-Pad1): track 0.00 -> 18.4 mm
- net /P2: track 0.00 -> 17.4 mm
- net Net-(BZ1-Pad1): track 0.00 -> 17.4 mm
- net Net-(Q3-Pad2): track 0.00 -> 16.9 mm
- net Net-(Q2-Pad2): track 0.00 -> 10.3 mm
- net Net-(Q2-Pad1): track 0.00 -> 5.62 mm
- net GND: track 0.00 -> 5.52 mm
- net Net-(D5-Pad1): track 0.00 -> 5.46 mm
- net Net-(D12-Pad2): track 0.00 -> 5.46 mm
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- added copper zone on F.Cu, net GND
Other:
- board outline added: 43 x 73 mm
