File: 25-station-led-alarm_v2/25-station-led-alarm.sch (KiCad schematic (older format))
At the start: 31 parts, among them J1 Conn_02x03_Counter_Clockwise, Q1 Q_NMOS_DGS, Q2 Q_NMOS_DGS, Q3 Q_NMOS_DGS

Commit message: gg
Parts:
- removed H1, H2, H3, H4: MountingHole_Pad, MountingHole:MountingHole_2.7mm_M2.5, symbol Mechanical:MountingHole_Pad
- removed J1: Conn_02x03_Counter_Clockwise, Connector_PinHeader_2.54mm:PinHeader_2x03_P2.54mm_Horizontal, symbol Connector_Generic:Conn_02x03_Counter_Clockwise
- added C?: 10uF, symbol Device:C_Small
- added J?: Conn_01x03_Female, symbol Connector:Conn_01x03_Female
- added J?: Conn_01x04_Female, symbol Connector:Conn_01x04_Female
- added R? (x2): R_sin 20k, Resistor_THT:R_Axial_DIN0309_L9.0mm_D3.2mm_P15.24mm_Horizontal, symbol Device:R_Small
- added R?: R_sin 1k, Resistor_THT:R_Axial_DIN0309_L9.0mm_D3.2mm_P15.24mm_Horizontal, symbol Device:R_Small
- added U?: OPAMP, symbol pspice:OPAMP
- added U?: 74LVC2G32, Package_DIP:DIP-14_W10.16mm, symbol 74xGxx:74LVC2G32
Connections:
- net labels added: signal
- net labels removed: P3, P4
- wire segments 59 -> 72
- no-connect marks 0 -> 2

Commit message: fe
Parts:
- removed BZ1: Buzzer, Buzzer_Beeper:resita_buzzer, symbol Device:Buzzer
- removed C?: 10uF, symbol Device:C_Small
- removed R1: R_sound 30, Resistor_THT:R_Axial_DIN0309_L9.0mm_D3.2mm_P15.24mm_Horizontal, symbol Device:R_Small
- removed R8: R_gate 10k, Resistor_THT:R_Axial_DIN0309_L9.0mm_D3.2mm_P15.24mm_Horizontal, symbol Device:R_Small
- removed R9: R_led 15, Resistor_THT:R_Axial_DIN0309_L9.0mm_D3.2mm_P12.70mm_Horizontal, symbol Device:R_Small
- removed R? (x2): R_sin 20k, Resistor_THT:R_Axial_DIN0309_L9.0mm_D3.2mm_P15.24mm_Horizontal, symbol Device:R_Small
- removed R?: R_sin 1k, Resistor_THT:R_Axial_DIN0309_L9.0mm_D3.2mm_P15.24mm_Horizontal, symbol Device:R_Small
- removed U?: OPAMP, symbol pspice:OPAMP
- removed U?: 74LVC2G32, Package_DIP:DIP-14_W10.16mm, symbol 74xGxx:74LVC2G32
- added J3, J4: Conn_01x02_Female, Connector_PinHeader_2.54mm:PinHeader_1x02_P2.54mm_Vertical, symbol Connector:Conn_01x02_Female
- added Q4: Q_NMOS_DGS, Package_TO_SOT_THT:TO-92, symbol Device:Q_NMOS_DGS
- J1: renamed from J?; footprint (none) -> Connector_PinHeader_2.54mm:PinHeader_1x04_P2.54mm_Vertical
- J2: renamed from J?; footprint (none) -> Connector_PinHeader_2.54mm:PinHeader_1x03_P2.54mm_Vertical
Connections:
- net +5V: now also J3.1 (Pin_1)
- net GND: now also Q4.3 (S)
- net at Q1.2 (G), R2.1, R4.1: now also Q4.2 (G)
- net at D13.1 (K): now also J3.2 (Pin_2), J4.1 (Pin_1)
- net at D13.2 (A), Q3.1 (D): now also J4.2 (Pin_2), Q4.1 (D)
- net at Q2.2 (G), R5.1, R7.1: now also Q3.2 (G)
Other:
- note removed: "sau dioda normala , \nde cercetat la nevoie"

Commit message: r
Parts:
- added C3: C_Small 47, Capacitor_THT:C_Rect_L9.0mm_W3.2mm_P7.50mm_MKT, symbol Device:C_Small
Connections:
- net +5V: now also C3.2
- net GND: now also C3.1
Changed lines of the file:
@@
 $EndComp
 Wire Wire Line
-	2650 5400 3000 5400
+	2650 5400 2900 5400
 Wire Wire Line
 	3000 4650 2800 4650
@@
 $EndComp
 Wire Wire Line
-	2850 5200 3000 5200
+	2850 5200 2900 5200
 $Comp
 L Connector:Conn_01x04_Female J1
@@
 Wire Wire Line
 	6400 2350 6400 2550
+$Comp
+L Device:C_Small C3
+U 1 1 619B2B9C
+P 2900 5300
+F 0 "C3" H 2992 5346 50  0000 L CNN
+F 1 "C_Small 47" H 2992 5255 50  0000 L CNN
+F 2 "Capacitor_THT:C_Rect_L9.0mm_W3.2mm_P7.50mm_MKT" H 2900 5300 50  0001 C CNN
+F 3 "~" H 2900 5300 50  0001 C CNN
+	1    2900 5300
+	1    0    0    -1
+$EndComp
+Connection ~ 2900 5200
+Wire Wire Line
+	2900 5200 3000 5200
+Connection ~ 2900 5400
+Wire Wire Line
+	2900 5400 3000 5400
 $EndSCHEMATC
