File: tests/tests.kicad_pcb (KiCad board)
At the start: 2 copper layers, 6 parts, among them U1 OP07, U2 OP07, U3 ESP32-WROOM-32

Commit message: f
Parts:
- added J2: Micro_SD_Card, Connector_Card:microSD_HC_Hirose_DM3D-SF, F.Cu at (142.2, 50.8)
- added J3: RJ45, Connector_RJ:RJ45_Amphenol_RJHSE538X, F.Cu at (272.5, 75.4)
- added J4: RJ45_Abracon_ARJP11A-MASA-B-A-EMU2, Connector_RJ:RJ45_Abracon_ARJP11A-MA_Horizontal, F.Cu at (262.3, 60.8)
- added J5: Wuerth_7499010121A, Connector_RJ:RJ45_Wuerth_7499010121A_Horizontal, F.Cu at (265.0, 23.7)
- added R3: 1000, Resistor_THT:R_Axial_DIN0204_L3.6mm_D1.6mm_P7.62mm_Horizontal, F.Cu at (151.1, 48.0)
- added R4: 5000, Resistor_THT:R_Axial_DIN0204_L3.6mm_D1.6mm_P7.62mm_Horizontal, F.Cu at (151.1, 44.9)
- added R5: R_Small, Resistor_THT:R_Axial_DIN0204_L3.6mm_D1.6mm_P7.62mm_Horizontal, F.Cu at (176.5, 37.4)
- added R6: R_Small, Resistor_THT:R_Axial_DIN0204_L3.6mm_D1.6mm_P7.62mm_Horizontal, F.Cu at (176.5, 27.9)
- added R7: R_Small, Resistor_THT:R_Axial_DIN0204_L3.6mm_D1.6mm_P7.62mm_Horizontal, F.Cu at (176.5, 31.1)
- added R8: R_Small, Resistor_THT:R_Axial_DIN0204_L3.6mm_D1.6mm_P7.62mm_Horizontal, F.Cu at (176.5, 34.2)
- added U4: ADA4841-1YRJ, Package_TO_SOT_SMD:SOT-23-6, F.Cu at (152.2, 51.8)
Connections:
- U1 pad 1: (no net) -> unconnected-(U1-Pad1)
- U1 pad 4: (no net) -> unconnected-(U1-Pad4)
- U1 pad 5: (no net) -> unconnected-(U1-Pad5)
- U1 pad 7: (no net) -> unconnected-(U1-Pad7)
- U1 pad 8: (no net) -> unconnected-(U1-Pad8)
- U2 pad 1: (no net) -> unconnected-(U2-Pad1)
- U2 pad 4: (no net) -> unconnected-(U2-Pad4)
- U2 pad 5: (no net) -> unconnected-(U2-Pad5)
- U2 pad 6: (no net) -> unconnected-(U2-Pad6)
- U2 pad 7: (no net) -> unconnected-(U2-Pad7)
- U2 pad 8: (no net) -> unconnected-(U2-Pad8)
- U3 pad 10: (no net) -> unconnected-(U3-Pad10)
- U3 pad 11: (no net) -> unconnected-(U3-Pad11)
- U3 pad 12: (no net) -> unconnected-(U3-Pad12)
- U3 pad 13: (no net) -> unconnected-(U3-Pad13)
- U3 pad 14: (no net) -> unconnected-(U3-Pad14)
- U3 pad 16: (no net) -> unconnected-(U3-Pad16)
- U3 pad 17: (no net) -> unconnected-(U3-Pad17)
- U3 pad 18: (no net) -> unconnected-(U3-Pad18)
- U3 pad 19: (no net) -> unconnected-(U3-Pad19)
- U3 pad 2: (no net) -> unconnected-(U3-Pad2)
- U3 pad 20: (no net) -> unconnected-(U3-Pad20)
- U3 pad 21: (no net) -> unconnected-(U3-Pad21)
- U3 pad 22: (no net) -> unconnected-(U3-Pad22)
- U3 pad 23: (no net) -> unconnected-(U3-Pad23)
- U3 pad 24: (no net) -> unconnected-(U3-Pad24)
- U3 pad 25: (no net) -> unconnected-(U3-Pad25)
- U3 pad 26: (no net) -> unconnected-(U3-Pad26)
- U3 pad 27: (no net) -> unconnected-(U3-Pad27)
- U3 pad 28: (no net) -> unconnected-(U3-Pad28)
- U3 pad 29: (no net) -> unconnected-(U3-Pad29)
- U3 pad 3: (no net) -> unconnected-(U3-Pad3)
- U3 pad 30: (no net) -> unconnected-(U3-Pad30)
- U3 pad 31: (no net) -> unconnected-(U3-Pad31)
- U3 pad 32: (no net) -> unconnected-(U3-Pad32)
- U3 pad 33: (no net) -> unconnected-(U3-Pad33)
- U3 pad 34: (no net) -> unconnected-(U3-Pad34)
- U3 pad 35: (no net) -> unconnected-(U3-Pad35)
- U3 pad 36: (no net) -> unconnected-(U3-Pad36)
- U3 pad 37: (no net) -> unconnected-(U3-Pad37)
- U3 pad 39: (no net) -> Net-(U3-Pad1)
- U3 pad 4: (no net) -> unconnected-(U3-Pad4)
- U3 pad 5: (no net) -> unconnected-(U3-Pad5)
- U3 pad 6: (no net) -> unconnected-(U3-Pad6)
- U3 pad 7: (no net) -> unconnected-(U3-Pad7)
- U3 pad 8: (no net) -> unconnected-(U3-Pad8)
- U3 pad 9: (no net) -> unconnected-(U3-Pad9)
Routing:
- net unconnected-(U3-Pad25): track 0.00 -> 82.9 mm
- net (no net): track 82.9 -> 0.00 mm
- net Net-(AE1-Pad1): track 21.3 -> 18.5 mm
Other:
- net class Default removed
