File: RPI_HAT_sensors/RPI_HAT_sensors.sch (KiCad schematic (older format))
At the start: 15 parts, among them J3 40HAT, U1 MQ135, U2 MQ137, U3 MQ136, U4 MCP3208, U5 LM4040LP-4.1

Commit message: y
Parts:
- added JP?: Jumper_2_Open, symbol Jumper:Jumper_2_Open
- added R?: 10k, Resistor_THT:R_Axial_DIN0204_L3.6mm_D1.6mm_P7.62mm_Horizontal, symbol Device:R_Small
- R1: value R_Small -> 1k; footprint (none) -> Resistor_THT:R_Axial_DIN0204_L3.6mm_D1.6mm_P7.62mm_Horizontal
- RV1, RV2, RV3: footprint (none) -> Potentiometer_THT:Potentiometer_Bourns_3339P_Vertical
Connections:
- net labels added: decider
- wire segments 67 -> 73
- no-connect marks 33 -> 32
Other:
- note added: "Pt a limita curentul la 2mA"
- note added: "circuit decizie cada referinta de precizie este prezenta cau nu"
- moved on the sheet: H1, H2, H3, H4, R1, RV1, RV2, RV3, U1, U2, U3, U4

Commit message: i
Parts:
- removed JP1: SolderJumper_3_Open, Jumper:SolderJumper-3_P1.3mm_Open_Pad1.0x1.5mm, symbol Jumper:SolderJumper_3_Open
- removed U5: LM4040LP-4.1, Package_TO_SOT_THT:TO-92_Inline, symbol Reference_Voltage:LM4040LP-4.1
- added C1: 10u, Capacitor_THT:C_Disc_D5.1mm_W3.2mm_P5.00mm, symbol Device:C_Small
- added C2: 1u, Capacitor_THT:C_Disc_D5.1mm_W3.2mm_P5.00mm, symbol Device:C_Small
- added J1: MOTOR, Connector_PinHeader_2.54mm:PinHeader_1x02_P2.54mm_Vertical, symbol Connector:Conn_01x02_Male
- added Q1: Q_NMOS_SGD, Package_TO_SOT_THT:TO-92, symbol Device:Q_NMOS_SGD
- added R2: 10k, Resistor_THT:R_Axial_DIN0204_L3.6mm_D1.6mm_P7.62mm_Horizontal, symbol Device:R_Small
- added R3: 5.1k, Resistor_THT:R_Axial_DIN0204_L3.6mm_D1.6mm_P7.62mm_Horizontal, symbol Device:R_Small
- added U5: DHT11, Sensor:Aosong_DHT11_5.5x12.0_P2.54mm, symbol Sensor:DHT11
- JP1: renamed from JP?; footprint (none) -> Connector_PinHeader_2.54mm:PinHeader_1x02_P2.54mm_Vertical
- R1: value 1k -> 220+
- gave numbers to parts that had none: 1
Connections:
- net labels added: DHT11, motor_control
- wire segments 73 -> 94
- no-connect marks 32 -> 30
Other:
- note removed: "Pt a limita curentul la 2mA"

Commit message: f
Parts:
- removed JP1: Jumper_2_Open, Connector_PinHeader_2.54mm:PinHeader_1x02_P2.54mm_Vertical, symbol Jumper:Jumper_2_Open
- added J2: MOTOR, Connector_PinHeader_2.54mm:PinHeader_1x02_P2.54mm_Vertical, symbol Connector:Conn_01x02_Male
- added Q2: Q_NMOS_SGD, Package_TO_SOT_THT:TO-92, symbol Device:Q_NMOS_SGD
- added R5: 10k, Resistor_THT:R_Axial_DIN0204_L3.6mm_D1.6mm_P7.62mm_Horizontal, symbol Device:R_Small
- R4: value 10k -> 220+
Connections:
- net +3V3: no longer R4.1
- net +5V: now also J2.1 (Pin_1)
- net ENABLE: now also J3.16 (BCM23); no longer J3.12 (BCM18)
- net GND: now also Q2.1 (S), R5.2
- net motor_control: now also J3.12 (BCM18); no longer J3.8 (BCM14)
- net motor_control2: now reaches J3.33 (BCM13)
- net motor_control2: now also R4.1
- net decider: no longer names the net of J3.36 (BCM16)
- net decider: no longer R4.2
- new net: J2.2 (Pin_2), Q2.3 (D)
- new net: Q2.2 (G), R4.2, R5.1
- no-connect marks 30 -> 29
Other:
- note added: "PWM0"
- note added: "PWM1"
- note removed: "circuit decizie cada referinta de precizie este prezenta cau nu"
- moved on the sheet: J1, Q1, R1, R2
Changed lines of the file:
@@
 Wire Wire Line
 	1650 3950 2000 3950
-Text Label 3350 2750 0    50   ~ 0
+Text Label 3350 2950 0    50   ~ 0
 ENABLE
 Wire Wire Line
-	3200 2750 3350 2750
+	3200 2950 3350 2950
 NoConn ~ 6200 9250
 NoConn ~ 6200 9350
@@
 NoConn ~ 2000 3650
 NoConn ~ 2000 3750
-NoConn ~ 2000 3850
 NoConn ~ 2000 4050
 NoConn ~ 3200 3750
@@
 NoConn ~ 3200 3250
 NoConn ~ 3200 3050
-NoConn ~ 3200 2950
 Wire Wire Line
 	6700 8700 6700 8750
-$Comp
-L Jumper:Jumper_2_Open JP1
-U 1 1 61C1D9B5
-P 11300 8800
-F 0 "JP1" V 11254 8898 50  0000 L CNN
-F 1 "Jumper_2_Open" V 11345 8898 50  0000 L CNN
-F 2 "Connector_PinHeader_2.54mm:PinHeader_1x02_P2.54mm_Vertical" H 11300 8800 50  0001 C CNN
-F 3 "~" H 11300 8800 50  0001 C CNN
-	1    11300 8800
-	0    1    1    0
-$EndComp
-Text Label 3350 3950 0    50   ~ 0
-decider
-Text Label 10700 8500 0    50   ~ 0
-decider
-Wire Wire Line
-	3200 3950 3350 3950
-$Comp
-L power:+3.3V #PWR0114
-U 1 1 61C223EE
-P 11300 8150
-F 0 "#PWR0114" H 11300 8000 50  0001 C CNN
-F 1 "+3.3V" H 11315 8323 50  0000 C CNN
-F 2 "" H 11300 8150 50  0001 C CNN
-F 3 "" H 11300 8150 50  0001 C CNN
-	1    11300 8150
-	1    0    0    -1
-$EndComp
-$Comp
-L power:GND #PWR0115
-U 1 1 61C23828
-P 11300 9050
-F 0 "#PWR0115" H 11300 8800 50  0001 C CNN
-F 1 "GND" H 11305 8877 50  0000 C CNN
-F 2 "" H 11300 9050 50  0001 C CNN
-F 3 "" H 11300 9050 50  0001 C CNN
-	1    11300 9050
-	1    0    0    -1
-$EndComp
-$Comp
-L Device:R_Small R4
-U 1 1 61C24B27
-P 11300 8300
-F 0 "R4" H 11359 8346 50  0000 L CNN
-F 1 "10k" H 11359 8255 50  0000 L CNN
-F 2 "Resistor_THT:R_Axial_DIN0204_L3.6mm_D1.6mm_P7.62mm_Horizontal" H 11300 8300 50  0001 C CNN
-F 3 "~" H 11300 8300 50  0001 C CNN
-	1    11300 8300
-	1    0    0    -1
-$EndComp
-Wire Wire Line
-	11300 9050 11300 9000
-Wire Wire Line
-	11300 8600 11300 8500
-Wire Wire Line
-	11300 8200 11300 8150
-Wire Wire Line
-	10700 8500 11300 8500
-Connection ~ 11300 8500
-Wire Wire Line
-	11300 8500 11300 8400
-Text Notes 11400 8600 0    50   ~ 0
-circuit decizie cada referinta de precizie este prezenta cau nu
 Wire Wire Line
 	11450 4400 11450 4500
@@
 Wire Wire Line
 	7000 8700 7000 8750
-Text Label 3350 2550 0    50   ~ 0
+Text Label 3350 2750 0    50   ~ 0
 motor_control
 Wire Wire Line
-	3350 2550 3200 2550
-Text Label 6200 6000 2    50   ~ 0
+	3350 2750 3200 2750
+Text Label 4600 6100 2    50   ~ 0
 motor_control
 $Comp
 L power:GND #PWR0116
 U 1 1 61C346B6
-P 6700 6700
-F 0 "#PWR0116" H 6700 6450 50  0001 C CNN
-F 1 "GND" H 6705 6527 50  0000 C CNN
-F 2 "" H 6700 6700 50  0001 C CNN
-F 3 "" H 6700 6700 50  0001 C CNN
-	1    6700 6700
+P 5100 6800
+F 0 "#PWR0116" H 5100 6550 50  0001 C CNN
+F 1 "GND" H 5105 6627 50  0000 C CNN
+F 2 "" H 5100 6800 50  0001 C CNN
+F 3 "" H 5100 6800 50  0001 C CNN
+	1    5100 6800
 	1    0    0    -1
 $EndComp
@@
 L power:+5V #PWR0117
 U 1 1 61C34FC9
-P 7150 5150
-F 0 "#PWR0117" H 7150 5000 50  0001 C CNN
-F 1 "+5V" H 7165 5323 50  0000 C CNN
-F 2 "" H 7150 5150 50  0001 C CNN
-F 3 "" H 7150 5150 50  0001 C CNN
-	1    7150 5150
+P 5550 5250
+F 0 "#PWR0117" H 5550 5100 50  0001 C CNN
+F 1 "+5V" H 5565 5423 50  0000 C CNN
+F 2 "" H 5550 5250 50  0001 C CNN
+F 3 "" H 5550 5250 50  0001 C CNN
+	1    5550 5250
 	1    0    0    -1
 $EndComp
@@
 L Connector:Conn_01x02_Male J1
 U 1 1 61C361D9
-P 6950 5500
-F 0 "J1" H 7058 5681 50  0000 C CNN
-F 1 "MOTOR" H 7058 5590 50  0000 C CNN
-F 2 "Connector_PinHeader_2.54mm:PinHeader_1x02_P2.54mm_Vertical" H 6950 5500 50  0001 C CNN
-F 3 "~" H 6950 5500 50  0001 C CNN
-	1    6950 5500
-	1    0    0    -1
-$EndComp
-Wire Wire Line
-	6200 6000 6350 6000
-Wire Wire Line
-	6550 6000 6700 6000
-Wire Wire Line
-	6700 6700 6700 6600
-Wire Wire Line
-	6700 6300 6700 6000
-Connection ~ 6700 6000
-Wire Wire Line
-	6700 6000 6850 6000
-Wire Wire Line
-	6700 6600 7150 6600
-Wire Wire Line
-	7150 6600 7150 6200
-Connection ~ 6700 6600
-Wire Wire Line
-	6700 6600 6700 6500
-Wire Wire Line
-	7150 5800 7150 5600
-Wire Wire Line
-	7150 5500 7150 5150
+P 5350 5600
+F 0 "J1" H 5458 5781 50  0000 C CNN
+F 1 "MOTOR" H 5458 5690 50  0000 C CNN
+F 2 "Connector_PinHeader_2.54mm:PinHeader_1x02_P2.54mm_Vertical" H 5350 5600 50  0001 C CNN
+F 3 "~" H 5350 5600 50  0001 C CNN
+	1    5350 5600
+	1    0    0    -1
+$EndComp
+Wire Wire Line
+	4600 6100 4750 6100
+Wire Wire Line
+	4950 6100 5100 6100
+Wire Wire Line
+	5100 6800 5100 6700
+Wire Wire Line
+	5100 6400 5100 6100
+Connection ~ 5100 6100
+Wire Wire Line
+	5100 6100 5250 6100
+Wire Wire Line
+	5100 6700 5550 6700
+Wire Wire Line
+	5550 6700 5550 6300
+Connection ~ 5100 6700
+Wire Wire Line
+	5100 6700 5100 6600
+Wire Wire Line
+	5550 5900 5550 5700
+Wire Wire Line
+	5550 5600 5550 5250
 $Comp
 L Device:Q_NMOS_SGD Q1
 U 1 1 61C457D4
-P 7050 6000
-F 0 "Q1" H 7256 6046 50  0000 L CNN
-F 1 "Q_NMOS_SGD" H 7256 5955 50  0000 L CNN
-F 2 "Package_TO_SOT_THT:TO-92" H 7250 6100 50  0001 C CNN
-F 3 "~" H 7050 6000 50  0001 C CNN
-	1    7050 6000
+P 5450 6100
+F 0 "Q1" H 5656 6146 50  0000 L CNN
+F 1 "Q_NMOS_SGD" H 5656 6055 50  0000 L CNN
+F 2 "Package_TO_SOT_THT:TO-92" H 5650 6200 50  0001 C CNN
+F 3 "~" H 5450 6100 50  0001 C CNN
+	1    5450 6100
 	1    0    0    -1
 $EndComp
@@
 L Device:R_Small R2
 U 1 1 61C70057
-P 6700 6400
-F 0 "R2" H 6759 6446 50  0000 L CNN
-F 1 "10k" H 6759 6355 50  0000 L CNN
-F 2 "Resistor_THT:R_Axial_DIN0204_L3.6mm_D1.6mm_P7.62mm_Horizontal" H 6700 6400 50  0001 C CNN
-F 3 "~" H 6700 6400 50  0001 C CNN
-	1    6700 6400
+P 5100 6500
+F 0 "R2" H 5159 6546 50  0000 L CNN
+F 1 "10k" H 5159 6455 50  0000 L CNN
+F 2 "Resistor_THT:R_Axial_DIN0204_L3.6mm_D1.6mm_P7.62mm_Horizontal" H 5100 6500 50  0001 C CNN
+F 3 "~" H 5100 6500 50  0001 C CNN
+	1    5100 6500
 	1    0    0    -1
 $EndComp
@@
 L Device:R_Small R1
 U 1 1 61C70D7E
-P 6450 6000
-F 0 "R1" H 6509 6046 50  0000 L CNN
-F 1 "220+" H 6509 5955 50  0000 L CNN
-F 2 "Resistor_THT:R_Axial_DIN0204_L3.6mm_D1.6mm_P7.62mm_Horizontal" H 6450 6000 50  0001 C CNN
-F 3 "~" H 6450 6000 50  0001 C CNN
-	1    6450 6000
+P 4850 6100
+F 0 "R1" H 4909 6146 50  0000 L CNN
+F 1 "220+" H 4909 6055 50  0000 L CNN
+F 2 "Resistor_THT:R_Axial_DIN0204_L3.6mm_D1.6mm_P7.62mm_Horizontal" H 4850 6100 50  0001 C CNN
+F 3 "~" H 4850 6100 50  0001 C CNN
+	1    4850 6100
 	0    -1   -1   0
 $EndComp
@@
 	0    -1   -1   0
 $EndComp
+Text Label 1850 3850 2    50   ~ 0
+motor_control2
+Wire Wire Line
+	1850 3850 2000 3850
+NoConn ~ 3200 3950
+Text Notes 1000 3850 0    50   ~ 0
+PWM1
+Text Notes 3900 2750 0    50   ~ 0
+PWM0
+Text Label 7150 6150 2    50   ~ 0
+motor_control2
+$Comp
+L power:GND #PWR0114
+U 1 1 61C65D18
+P 7650 6850
+F 0 "#PWR0114" H 7650 6600 50  0001 C CNN
+F 1 "GND" H 7655 6677 50  0000 C CNN
+F 2 "" H 7650 6850 50  0001 C CNN
+F 3 "" H 7650 6850 50  0001 C CNN
+	1    7650 6850
+	1    0    0    -1
+$EndComp
+$Comp
+L power:+5V #PWR0115
+U 1 1 61C65D1E
+P 8100 5300
+F 0 "#PWR0115" H 8100 5150 50  0001 C CNN
+F 1 "+5V" H 8115 5473 50  0000 C CNN
+F 2 "" H 8100 5300 50  0001 C CNN
+F 3 "" H 8100 5300 50  0001 C CNN
+	1    8100 5300
+	1    0    0    -1
+$EndComp
+$Comp
+L Connector:Conn_01x02_Male J2
+U 1 1 61C65D24
+P 7900 5650
+F 0 "J2" H 8008 5831 50  0000 C CNN
+F 1 "MOTOR" H 8008 5740 50  0000 C CNN
+F 2 "Connector_PinHeader_2.54mm:PinHeader_1x02_P2.54mm_Vertical" H 7900 5650 50  0001 C CNN
+F 3 "~" H 7900 5650 50  0001 C CNN
+	1    7900 5650
+	1    0    0    -1
+$EndComp
+Wire Wire Line
+	7150 6150 7300 6150
+Wire Wire Line
+	7500 6150 7650 6150
+Wire Wire Line
+	7650 6850 7650 6750
+Wire Wire Line
+	7650 6450 7650 6150
+Connection ~ 7650 6150
+Wire Wire Line
+	7650 6150 7800 6150
+Wire Wire Line
+	7650 6750 8100 6750
+Wire Wire Line
+	8100 6750 8100 6350
+Connection ~ 7650 6750
+Wire Wire Line
+	7650 6750 7650 6650
+Wire Wire Line
+	8100 5950 8100 5750
+Wire Wire Line
+	8100 5650 8100 5300
+$Comp
+L Device:Q_NMOS_SGD Q2
+U 1 1 61C65D36
+P 8000 6150
+F 0 "Q2" H 8206 6196 50  0000 L CNN
+F 1 "Q_NMOS_SGD" H 8206 6105 50  0000 L CNN
+F 2 "Package_TO_SOT_THT:TO-92" H 8200 6250 50  0001 C CNN
+F 3 "~" H 8000 6150 50  0001 C CNN
+	1    8000 6150
+	1    0    0    -1
+$EndComp
+$Comp
+L Device:R_Small R5
+U 1 1 61C65D3C
+P 7650 6550
+F 0 "R5" H 7709 6596 50  0000 L CNN
+F 1 "10k" H 7709 6505 50  0000 L CNN
+F 2 "Resistor_THT:R_Axial_DIN0204_L3.6mm_D1.6mm_P7.62mm_Horizontal" H 7650 6550 50  0001 C CNN
+F 3 "~" H 7650 6550 50  0001 C CNN
+	1    7650 6550
+	1    0    0    -1
+$EndComp
+$Comp
+L Device:R_Small R4
+U 1 1 61C65D42
+P 7400 6150
+F 0 "R4" H 7459 6196 50  0000 L CNN
+F 1 "220+" H 7459 6105 50  0000 L CNN
+F 2 "Resistor_THT:R_Axial_DIN0204_L3.6mm_D1.6mm_P7.62mm_Horizontal" H 7400 6150 50  0001 C CNN
+F 3 "~" H 7400 6150 50  0001 C CNN
+	1    7400 6150
+	0    -1   -1   0
+$EndComp

Commit message: prod files
Parts:
- added FID1, FID2, FID3: Fiducial, Fiducial:Fiducial_1.5mm_Mask3mm, symbol Mechanical:Fiducial
Changed lines of the file:
@@
 	0    -1   -1   0
 $EndComp
+$Comp
+L Mechanical:Fiducial FID3
+U 1 1 61C8CBCA
+P 2450 9050
+F 0 "FID3" H 2535 9096 50  0000 L CNN
+F 1 "Fiducial" H 2535 9005 50  0000 L CNN
+F 2 "Fiducial:Fiducial_1.5mm_Mask3mm" H 2450 9050 50  0001 C CNN
+F 3 "~" H 2450 9050 50  0001 C CNN
+	1    2450 9050
+	1    0    0    -1
+$EndComp
+$Comp
+L Mechanical:Fiducial FID2
+U 1 1 61C8D70B
+P 1950 9050
+F 0 "FID2" H 2035 9096 50  0000 L CNN
+F 1 "Fiducial" H 2035 9005 50  0000 L CNN
+F 2 "Fiducial:Fiducial_1.5mm_Mask3mm" H 1950 9050 50  0001 C CNN
+F 3 "~" H 1950 9050 50  0001 C CNN
+	1    1950 9050
+	1    0    0    -1
+$EndComp
+$Comp
+L Mechanical:Fiducial FID1
+U 1 1 61C8DD5E
+P 1450 9050
+F 0 "FID1" H 1535 9096 50  0000 L CNN
+F 1 "Fiducial" H 1535 9005 50  0000 L CNN
+F 2 "Fiducial:Fiducial_1.5mm_Mask3mm" H 1450 9050 50  0001 C CNN
+F 3 "~" H 1450 9050 50  0001 C CNN
+	1    1450 9050
+	1    0    0    -1
+$EndComp
 $EndSCHEMATC

Commit message: ff
Parts:
- added C3: 1u, Capacitor_THT:C_Disc_D5.1mm_W3.2mm_P5.00mm, symbol Device:C_Small
- added JP1: Jumper_2_Open, Connector_PinHeader_2.54mm:PinHeader_1x02_P2.54mm_Vertical, symbol Jumper:Jumper_2_Open
- added R6, R7, R8: 3K9, Resistor_THT:R_Axial_DIN0204_L3.6mm_D1.6mm_P7.62mm_Horizontal, symbol Device:R_Small
- added U6: CAT24C32-raspberrypi_hat, Package_SO:TSSOP-8_4.4x3mm_P0.65mm, symbol RPI_HAT_sensors-rescue:CAT24C32-raspberrypi_hat
Connections:
- net +3V3: now also C3.2, R6.2, R7.1, R8.1, U6.8 (VCC)
- net GND: now also C3.1, JP1.1 (A), U6.1 (A0), U6.2 (A1), U6.3 (A2), U6.4 (GND)
- net EEPROM_SD: now reaches J3.27 (BCM0)
- net EEPROM_SD: now also R8.2, U6.5 (SDA)
- net EEPROM_SC: now reaches J3.28 (BCM1)
- net EEPROM_SC: now also R7.2, U6.6 (SCL)
- new net: JP1.2 (B), R6.1, U6.7 (WP)
- no-connect marks 29 -> 28
Other:
- moved on the sheet: C1, C2, FID1, FID2, FID3, H1, H2, H3, H4, J1, J2, Q1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

Commit message: f
Parts:
- added C4, C5, C6: 1u, Capacitor_SMD:C_0805_2012Metric_Pad1.15x1.40mm_HandSolder, symbol Device:C_Small
Connections:
- net ADC1: now also C6.2
- net ADC2: now also C5.2
- net ADC3: now also C4.2
- net GND: now also C4.1, C5.1, C6.1
Other:
- note added: "ADC"
- note added: "EEPROM"
- note added: "MOTOR CONTROL"
- note added: "SENSORS"
- moved on the sheet: C3, J1, J2, JP1, Q1, Q2, R1, R2, R3, R4, R5, R6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
