File: RPI_HAT_sensors/RPI_HAT_sensors.kicad_pcb (KiCad board)
At the start: 4 copper layers, 65 x 56 mm, 11 parts, among them J3 40HAT, U1 MQ135, U2 MQ137, U3 MQ136, U4 MCP3208, U5 LM4040LP-4.1

Commit message: y
Parts:
- added R1: 1k, Resistor_THT:R_Axial_DIN0204_L3.6mm_D1.6mm_P7.62mm_Horizontal, F.Cu at (106.7, 78.7)
- added RV1: R_POT, Potentiometer_THT:Potentiometer_Bourns_3339P_Vertical, F.Cu at (83.8, 97.7)
- added RV2: R_POT, Potentiometer_THT:Potentiometer_Bourns_3339P_Vertical, F.Cu at (92.9, 107.6)
- added RV3: R_POT, Potentiometer_THT:Potentiometer_Bourns_3339P_Vertical, F.Cu at (129.5, 110.9)
- moved U1 11.1 mm to (91.4, 81.1)
- moved U2 3.25 mm to (131.5, 96.2)
- moved U5 1.50 mm to (111.8, 72.6)
Routing:
- added copper zone on F.Cu, net +5V
- added copper zone on B.Cu, net GND
Changed lines of the file:
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@@
     (tracks 0)
     (zones 0)
-    (modules 11)
+    (modules 15)
     (nets 13)
   )
@@
   )
   (module Package_TO_SOT_THT:TO-92_Inline (layer F.Cu)
-    (at 113.23574 72.39 90)
+    (at 111.76 72.644 90)
     (descr "TO-92 leads in-line, narrow, oval pads, drill 0.75mm (see NXP sot054_po.pdf)")
     (tags "to-92 sc-43 sc-43a sot54 PA33 transistor")
@@
   )
   (module BEIA_sensors:MQ135 (layer F.Cu)
-    (at 90.06332 92.18422)
+    (at 91.44 81.11998)
     (fp_text reference U1 (at 0.4826 -1.6002) (layer F.SilkS)
       (effects (font (size 1 1) (thickness 0.15)))
@@
   )
   (module BEIA_sensors:MQ135 (layer F.Cu)
-    (at 131.75488 99.42322)
+    (at 131.45262 96.18726)
     (fp_text reference U2 (at 0.4826 -1.6002) (layer F.SilkS)
       (effects (font (size 1 1) (thickness 0.15)))
@@
       (net 2 +5V))
     (model ${KISYS3DMOD}/Package_DIP.3dshapes/DIP-16_W7.62mm.wrl
+      (at (xyz 0 0 0))
+      (scale (xyz 1 1 1))
+      (rotate (xyz 0 0 0))
+    )
+  )
+  (module Resistor_THT:R_Axial_DIN0204_L3.6mm_D1.6mm_P7.62mm_Horizontal (layer F.Cu)
+    (at 106.68 78.74 90)
+    (descr "Resistor, Axial_DIN0204 series, Axial, Horizontal, pin pitch=7.62mm, 0.167W, length*diameter=3.6*1.6mm^2, http://cdn-reichelt.de/documents/datenblatt/B400/1_4W%23YAG.pdf")
+    (tags "Resistor Axial_DIN0204 series Axial Horizontal pin pitch 7.62mm 0.167W length 3.6mm diameter 1.6mm")
+    (fp_text reference R1 (at 3.81 -1.92 90) (layer F.SilkS)
+      (effects (font (size 1 1) (thickness 0.15)))
+    )
+    (fp_text value 1k (at 3.81 1.92 90) (layer F.Fab)
+      (effects (font (size 1 1) (thickness 0.15)))
+    )
+    (fp_line (start 2.01 -0.8) (end 2.01 0.8) (layer F.Fab) (width 0.1))
+    (fp_line (start 2.01 0.8) (end 5.61 0.8) (layer F.Fab) (width 0.1))
+    (fp_line (start 5.61 0.8) (end 5.61 -0.8) (layer F.Fab) (width 0.1))
+    (fp_line (start 5.61 -0.8) (end 2.01 -0.8) (layer F.Fab) (width 0.1))
+    (fp_line (start 0 0) (end 2.01 0) (layer F.Fab) (width 0.1))
+    (fp_line (start 7.62 0) (end 5.61 0) (layer F.Fab) (width 0.1))
+    (fp_line (start 1.89 -0.92) (end 1.89 0.92) (layer F.SilkS) (width 0.12))
+    (fp_line (start 1.89 0.92) (end 5.73 0.92) (layer F.SilkS) (width 0.12))
+    (fp_line (start 5.73 0.92) (end 5.73 -0.92) (layer F.SilkS) (width 0.12))
+    (fp_line (start 5.73 -0.92) (end 1.89 -0.92) (layer F.SilkS) (width 0.12))
+    (fp_line (start 0.94 0) (end 1.89 0) (layer F.SilkS) (width 0.12))
+    (fp_line (start 6.68 0) (end 5.73 0) (layer F.SilkS) (width 0.12))
+    (fp_line (start -0.95 -1.05) (end -0.95 1.05) (layer F.CrtYd) (width 0.05))
+    (fp_line (start -0.95 1.05) (end 8.57 1.05) (layer F.CrtYd) (width 0.05))
+    (fp_line (start 8.57 1.05) (end 8.57 -1.05) (layer F.CrtYd) (width 0.05))
+    (fp_line (start 8.57 -1.05) (end -0.95 -1.05) (layer F.CrtYd) (width 0.05))
+    (fp_text user %R (at 3.81 0 90) (layer F.Fab)
+      (effects (font (size 0.72 0.72) (thickness 0.108)))
+    )
+    (pad 1 thru_hole circle (at 0 0 90) (size 1.4 1.4) (drill 0.7) (layers *.Cu *.Mask)
+      (net 2 +5V))
+    (pad 2 thru_hole oval (at 7.62 0 90) (size 1.4 1.4) (drill 0.7) (layers *.Cu *.Mask)
+      (net 12 "Net-(JP1-Pad1)"))
+    (model ${KISYS3DMOD}/Resistor_THT.3dshapes/R_Axial_DIN0204_L3.6mm_D1.6mm_P7.62mm_Horizontal.wrl
+      (at (xyz 0 0 0))
+      (scale (xyz 1 1 1))
+      (rotate (xyz 0 0 0))
+    )
+  )
+  (module Potentiometer_THT:Potentiometer_Bourns_3339P_Vertical (layer F.Cu)
+    (at 83.82 97.67316 270)
+    (descr "Potentiometer, vertical, Bourns 3339P, http://www.bourns.com/docs/Product-Datasheets/3339.pdf")
+    (tags "Potentiometer vertical Bourns 3339P")
+    (fp_text reference RV1 (at 0 -7.6 270) (layer F.SilkS)
+      (effects (font (size 1 1) (thickness 0.15)))
+    )
+    (fp_text value R_POT (at 0 2.52 270) (layer F.Fab)
+      (effects (font (size 1 1) (thickness 0.15)))
+    )
+    (fp_circle (center 0 -2.54) (end 3.81 -2.54) (layer F.Fab) (width 0.1))
+    (fp_circle (center 0 -2.54) (end 2.5 -2.54) (layer F.Fab) (width 0.1))
+    (fp_circle (center 0 -2.54) (end 3.93 -2.54) (layer F.SilkS) (width 0.12))
+    (fp_line (start 0 -0.064) (end 0.001 -5.014) (layer F.Fab) (width 0.1))
+    (fp_line (start 0 -0.064) (end 0.001 -5.014) (layer F.Fab) (width 0.1))
+    (fp_line (start -4.1 -6.6) (end -4.1 1.55) (layer F.CrtYd) (width 0.05))
+    (fp_line (start -4.1 1.55) (end 4.1 1.55) (layer F.CrtYd) (width 0.05))
+    (fp_line (start 4.1 1.55) (end 4.1 -6.6) (layer F.CrtYd) (width 0.05))
+    (fp_line (start 4.1 -6.6) (end -4.1 -6.6) (layer F.CrtYd) (width 0.05))
+    (fp_text user %R (at -3.018 -2.54) (layer F.Fab)
+      (effects (font (size 0.66 0.66) (thickness 0.15)))
+    )
+    (pad 3 thru_hole circle (at 0 -5.08 270) (size 1.26 1.26) (drill 0.7) (layers *.Cu *.Mask)
+      (net 1 GND))
+    (pad 2 thru_hole circle (at -2.54 -2.54 270) (size 1.26 1.26) (drill 0.7) (layers *.Cu *.Mask))
+    (pad 1 thru_hole circle (at 0 0 270) (size 1.26 1.26) (drill 0.7) (layers *.Cu *.Mask)
+      (net 7 /ADC1))
+    (model ${KISYS3DMOD}/Potentiometer_THT.3dshapes/Potentiometer_Bourns_3339P_Vertical.wrl
+      (at (xyz 0 0 0))
+      (scale (xyz 1 1 1))
+      (rotate (xyz 0 0 0))
+    )
+  )
+  (module Potentiometer_THT:Potentiometer_Bourns_3339P_Vertical (layer F.Cu)
+    (at 92.91066 107.56646 180)
+    (descr "Potentiometer, vertical, Bourns 3339P, http://www.bourns.com/docs/Product-Datasheets/3339.pdf")
+    (tags "Potentiometer vertical Bourns 3339P")
+    (fp_text reference RV2 (at 0 -7.6 180) (layer F.SilkS)
+      (effects (font (size 1 1) (thickness 0.15)))
+    )
+    (fp_text value R_POT (at 0 2.52 180) (layer F.Fab)
+      (effects (font (size 1 1) (thickness 0.15)))
+    )
+    (fp_text user %R (at -3.018 -2.54 270) (layer F.Fab)
+      (effects (font (size 0.66 0.66) (thickness 0.15)))
+    )
+    (fp_line (start 4.1 -6.6) (end -4.1 -6.6) (layer F.CrtYd) (width 0.05))
+    (fp_line (start 4.1 1.55) (end 4.1 -6.6) (layer F.CrtYd) (width 0.05))
+    (fp_line (start -4.1 1.55) (end 4.1 1.55) (layer F.CrtYd) (width 0.05))
+    (fp_line (start -4.1 -6.6) (end -4.1 1.55) (layer F.CrtYd) (width 0.05))
+    (fp_line (start 0 -0.064) (end 0.001 -5.014) (layer F.Fab) (width 0.1))
+    (fp_line (start 0 -0.064) (end 0.001 -5.014) (layer F.Fab) (width 0.1))
+    (fp_circle (center 0 -2.54) (end 3.93 -2.54) (layer F.SilkS) (width 0.12))
+    (fp_circle (center 0 -2.54) (end 2.5 -2.54) (layer F.Fab) (width 0.1))
+    (fp_circle (center 0 -2.54) (end 3.81 -2.54) (layer F.Fab) (width 0.1))
+    (pad 1 thru_hole circle (at 0 0 180) (size 1.26 1.26) (drill 0.7) (layers *.Cu *.Mask)
+      (net 9 /ADC2))
+    (pad 2 thru_hole circle (at -2.54 -2.54 180) (size 1.26 1.26) (drill 0.7) (layers *.Cu *.Mask))
+    (pad 3 thru_hole circle (at 0 -5.08 180) (size 1.26 1.26) (drill 0.7) (layers *.Cu *.Mask)
+      (net 1 GND))
+    (model ${KISYS3DMOD}/Potentiometer_THT.3dshapes/Potentiometer_Bourns_3339P_Vertical.wrl
+      (at (xyz 0 0 0))
+      (scale (xyz 1 1 1))
+      (rotate (xyz 0 0 0))
+    )
+  )
+  (module Potentiometer_THT:Potentiometer_Bourns_3339P_Vertical (layer F.Cu)
+    (at 129.54 110.91418 90)
+    (descr "Potentiometer, vertical, Bourns 3339P, http://www.bourns.com/docs/Product-Datasheets/3339.pdf")
+    (tags "Potentiometer vertical Bourns 3339P")
+    (fp_text reference RV3 (at 0 -7.6 90) (layer F.SilkS)
+      (effects (font (size 1 1) (thickness 0.15)))
+    )
+    (fp_text value R_POT (at 0 2.52 90) (layer F.Fab)
+      (effects (font (size 1 1) (thickness 0.15)))
+    )
+    (fp_circle (center 0 -2.54) (end 3.81 -2.54) (layer F.Fab) (width 0.1))
+    (fp_circle (center 0 -2.54) (end 2.5 -2.54) (layer F.Fab) (width 0.1))
+    (fp_circle (center 0 -2.54) (end 3.93 -2.54) (layer F.SilkS) (width 0.12))
+    (fp_line (start 0 -0.064) (end 0.001 -5.014) (layer F.Fab) (width 0.1))
+    (fp_line (start 0 -0.064) (end 0.001 -5.014) (layer F.Fab) (width 0.1))
+    (fp_line (start -4.1 -6.6) (end -4.1 1.55) (layer F.CrtYd) (width 0.05))
+    (fp_line (start -4.1 1.55) (end 4.1 1.55) (layer F.CrtYd) (width 0.05))
+    (fp_line (start 4.1 1.55) (end 4.1 -6.6) (layer F.CrtYd) (width 0.05))
+    (fp_line (start 4.1 -6.6) (end -4.1 -6.6) (layer F.CrtYd) (width 0.05))
+    (fp_text user %R (at -3.018 -2.54 180) (layer F.Fab)
+      (effects (font (size 0.66 0.66) (thickness 0.15)))
+    )
+    (pad 3 thru_hole circle (at 0 -5.08 90) (size 1.26 1.26) (drill 0.7) (layers *.Cu *.Mask)
+      (net 1 GND))
+    (pad 2 thru_hole circle (at -2.54 -2.54 90) (size 1.26 1.26) (drill 0.7) (layers *.Cu *.Mask))
+    (pad 1 thru_hole circle (at 0 0 90) (size 1.26 1.26) (drill 0.7) (layers *.Cu *.Mask)
+      (net 8 /ADC3))
+    (model ${KISYS3DMOD}/Potentiometer_THT.3dshapes/Potentiometer_Bourns_3339P_Vertical.wrl
       (at (xyz 0 0 0))
       (scale (xyz 1 1 1))
@@
       )
     )
+  )
+  (zone (net 2) (net_name +5V) (layer F.Cu) (hatch edge 0.508)
+    (connect_pads (clearance 0.2))
+    (min_thickness 0.254)
+    (fill yes (arc_segments 32) (thermal_gap 0.508) (thermal_bridge_width 0.508))
+    (polygon
+      (pts
+        (xy 78.99654 64.92748) (xy 78.99654 113.5507) (xy 81.81086 116.36502) (xy 139.71524 116.36502) (xy 143.17472 112.90554)
+        (xy 143.17472 64.83858) (xy 139.69238 61.35624) (xy 82.08264 61.35624)
+      )
+    )
+  )
+  (zone (net 1) (net_name GND) (layer B.Cu) (hatch edge 0.508)
+    (connect_pads (clearance 0.2))
+    (min_thickness 0.254)
+    (fill yes (arc_segments 32) (thermal_gap 0.508) (thermal_bridge_width 0.508))
+    (polygon
+      (pts
+        (xy 82.07502 61.3537) (xy 78.94066 64.48806) (xy 78.94066 113.5634) (xy 81.69656 116.3193) (xy 139.80668 116.3193)
+        (xy 143.11884 113.00714) (xy 143.11884 64.99098) (xy 139.49934 61.37148) (xy 139.4968 61.36894)
+      )
+    )

Commit message: i
Parts:
- added C1: 10u, Capacitor_THT:C_Disc_D5.1mm_W3.2mm_P5.00mm, F.Cu at (140.9, 69.5)
- added C2: 1u, Capacitor_THT:C_Disc_D5.1mm_W3.2mm_P5.00mm, F.Cu at (140.9, 81.9)
- added J1: MOTOR, Connector_PinHeader_2.54mm:PinHeader_1x02_P2.54mm_Vertical, F.Cu at (81.3, 71.1)
- added Q1: Q_NMOS_SGD, Package_TO_SOT_THT:TO-92, F.Cu at (86.4, 71.1)
- added R2: 10k, Resistor_THT:R_Axial_DIN0204_L3.6mm_D1.6mm_P7.62mm_Horizontal, F.Cu at (91.4, 73.7)
- added R3: 5.1k, Resistor_THT:R_Axial_DIN0204_L3.6mm_D1.6mm_P7.62mm_Horizontal, F.Cu at (111.5, 71.1)
- added R4: 10k, Resistor_THT:R_Axial_DIN0204_L3.6mm_D1.6mm_P7.62mm_Horizontal, F.Cu at (103.9, 73.7)
- JP1: value SolderJumper_3_Open -> Jumper_2_Open; footprint Jumper:SolderJumper-3_P1.3mm_Open_Pad1.0x1.5mm -> Connector_PinHeader_2.54mm:PinHeader_1x02_P2.54mm_Vertical
- R1: value 1k -> 220+
- U5: value LM4040LP-4.1 -> DHT11; footprint Package_TO_SOT_THT:TO-92_Inline -> Sensor:Aosong_DHT11_5.5x12.0_P2.54mm
- moved U5 18.1 mm to (111.0, 90.7), turned to 180 degrees
- moved JP1 11.8 mm to (109.7, 78.0), turned to 90 degrees
- moved R1 10.8 mm to (99.1, 71.1), turned to 180 degrees
- moved U1 8.14 mm to (95.7, 88.1)
- moved U4 3.64 mm to (119.4, 78.7)
- moved U2 2.82 mm to (130.4, 93.6), turned to 270 degrees
- moved RV3 1.72 mm to (129.5, 109.2)
- moved RV2 0.92 mm to (93.8, 107.3)
- moved U3 0.63 mm to (109.7, 105.0), turned to 90 degrees
- moved RV1 0.24 mm to (84.0, 97.6), turned to 180 degrees
Connections:
- J3 pad 1: (no net) -> +3V3
- J3 pad 10: (no net) -> /DHT11
- J3 pad 36: (no net) -> /decider
- J3 pad 8: (no net) -> /motor_control
- JP1 pad 1: Net-(JP1-Pad1) -> /decider
- JP1 pad 2: Net-(JP1-Pad2) -> GND
- R1 pad 1: +5V -> /motor_control
- R1 pad 2: Net-(JP1-Pad1) -> Net-(Q1-Pad2)
- RV1 pad 2: (no net) -> GND
- RV1 pad 3: GND -> (no net)
- RV2 pad 2: (no net) -> GND
- RV2 pad 3: GND -> (no net)
- RV3 pad 2: (no net) -> GND
- RV3 pad 3: GND -> (no net)
- U2 pad 5: (no net) -> GND
- U3 pad 2: Net-(U3-Pad2) -> +5V
- U3 pad 3: Net-(U3-Pad2) -> +5V
- U4 pad 15: Net-(JP1-Pad2) -> +5V
- U5 pad 1: (no net) -> +5V
- U5 pad 2: Net-(JP1-Pad1) -> /DHT11
- U5 pad 3: GND -> (no net)
Routing:
- net GND: track 0.00 -> 219.8 mm, vias 0 -> 1
- net +5V: track 0.00 -> 164.0 mm, vias 0 -> 1
- net /ADC2: track 0.00 -> 56.7 mm
- net /ADC1: track 0.00 -> 52.9 mm
- net /ADC3: track 0.00 -> 48.0 mm
- net /ENABLE: track 0.00 -> 43.8 mm
- net /DHT11: track 0.00 -> 31.9 mm
- net /decider: track 0.00 -> 29.2 mm
- net +3V3: track 0.00 -> 22.4 mm
- net /CLK: track 0.00 -> 16.6 mm
- net /motor_control: track 0.00 -> 9.94 mm
- net /DIN: track 0.00 -> 9.23 mm
- net Net-(Q1-Pad2): track 0.00 -> 6.88 mm
- net /DOUT: track 0.00 -> 5.76 mm
- net Net-(J1-Pad2): track 0.00 -> 5.08 mm
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
Commit message: f
Parts:
- removed JP1: Jumper_2_Open, Connector_PinHeader_2.54mm:PinHeader_1x02_P2.54mm_Vertical
- added J2: MOTOR, Connector_PinHeader_2.54mm:PinHeader_1x02_P2.54mm_Vertical, F.Cu at (140.8, 103.7)
- added Q2: Q_NMOS_SGD, Package_TO_SOT_THT:TO-92, F.Cu at (134.2, 107.0)
- added R5: 10k, Resistor_THT:R_Axial_DIN0204_L3.6mm_D1.6mm_P7.62mm_Horizontal, F.Cu at (135.4, 114.6)
- R4: value 10k -> 220+
- moved R4 3.05 mm to (103.9, 76.7)
- moved RV3 1.62 mm to (127.9, 108.7)
Connections:
- J3 pad 1: +3V3 -> (no net)
- J3 pad 12: /ENABLE -> /motor_control
- J3 pad 16: (no net) -> /ENABLE
- J3 pad 33: (no net) -> /motor_control2
- J3 pad 36: /decider -> (no net)
- J3 pad 8: /motor_control -> (no net)
- R4 pad 1: +3V3 -> /motor_control2
- R4 pad 2: /decider -> Net-(Q2-Pad2)
Routing:
- net Net-(Q2-Pad2): track 0.00 -> 62.3 mm, vias 0 -> 1
- net /motor_control2: track 0.00 -> 29.3 mm
- net /decider: track 29.2 -> 0.00 mm
- net +3V3: track 22.4 -> 0.00 mm
- net GND: track 219.8 -> 233.1 mm
- net +5V: track 164.0 -> 173.8 mm
- net Net-(J2-Pad2): track 0.00 -> 4.36 mm
- net /ENABLE: track 43.8 -> 41.4 mm
- net /motor_control: track 9.94 -> 8.77 mm
- net /ADC3: track 48.0 -> 47.4 mm
- net (no net): vias 66 -> 71
Other:
- board text added: "5V"

Commit message: prod files
Parts:
- added FID1: Fiducial, Fiducial:Fiducial_1.5mm_Mask3mm, F.Cu at (81.5, 84.8)
- added FID2: Fiducial, Fiducial:Fiducial_1.5mm_Mask3mm, F.Cu at (86.4, 110.2)
- added FID3: Fiducial, Fiducial:Fiducial_1.5mm_Mask3mm, F.Cu at (119.4, 114.0)

Commit message: ff
Parts:
- added C3: 1u, Capacitor_THT:C_Disc_D5.1mm_W3.2mm_P5.00mm, F.Cu at (109.6, 82.7)
- added JP1: Jumper_2_Open, Connector_PinHeader_2.54mm:PinHeader_1x02_P2.54mm_Vertical, F.Cu at (87.6, 75.7)
- added R6: 3K9, Resistor_THT:R_Axial_DIN0204_L3.6mm_D1.6mm_P7.62mm_Horizontal, F.Cu at (93.2, 74.3)
- added R7: 3K9, Resistor_THT:R_Axial_DIN0204_L3.6mm_D1.6mm_P7.62mm_Horizontal, F.Cu at (113.4, 77.4)
- added R8: 3K9, Resistor_THT:R_Axial_DIN0204_L3.6mm_D1.6mm_P7.62mm_Horizontal, F.Cu at (115.7, 77.4)
- added U6: CAT24C32-raspberrypi_hat, Package_SO:TSSOP-8_4.4x3mm_P0.65mm, F.Cu at (114.4, 90.8)
- moved FID1 19.9 mm to (92.0, 101.8)
- moved U5 7.10 mm to (103.9, 90.0)
- moved U1 6.03 mm to (89.7, 88.6)
- moved RV1 4.42 mm to (84.1, 102.0)
- moved FID2 3.63 mm to (87.2, 113.8)
- moved J1 2.44 mm to (83.0, 69.4)
- moved Q1 2.44 mm to (88.1, 69.4)
- moved R1 2.44 mm to (100.8, 69.4)
- moved R2 2.44 mm to (93.2, 72.0)
- moved R4 1.44 mm to (102.5, 76.9)
Connections:
- J3 pad 1: (no net) -> +3V3
- J3 pad 27: (no net) -> /EEPROM_SD
- J3 pad 28: (no net) -> /EEPROM_SC
Routing:
- net +5V: track 173.8 -> 116.5 mm, vias 1 -> 0
- net GND: track 233.1 -> 283.2 mm, vias 1 -> 5
- net +3V3: track 0.00 -> 48.3 mm
- net Net-(JP1-Pad2): track 0.00 -> 37.7 mm, vias 0 -> 1
- net /EEPROM_SC: track 0.00 -> 29.2 mm, vias 0 -> 1
- net /EEPROM_SD: track 0.00 -> 24.9 mm, vias 0 -> 1
- net Net-(Q2-Pad2): track 62.3 -> 51.7 mm, vias 1 -> 2
- net /motor_control2: track 29.3 -> 33.8 mm
- net /ADC1: track 52.9 -> 56.1 mm
- net /DHT11: track 31.9 -> 34.1 mm, vias 0 -> 1
- net /motor_control: track 8.77 -> 6.86 mm
- net (no net): vias 71 -> 52

Commit message: f
Parts:
- added C4: 1u, Capacitor_SMD:C_0805_2012Metric_Pad1.15x1.40mm_HandSolder, F.Cu at (125.8, 82.3)
- added C5: 1u, Capacitor_SMD:C_0805_2012Metric_Pad1.15x1.40mm_HandSolder, F.Cu at (121.7, 83.0)
- added C6: 1u, Capacitor_SMD:C_0805_2012Metric_Pad1.15x1.40mm_HandSolder, F.Cu at (118.4, 87.4)
Routing:
- net GND: track 283.2 -> 292.3 mm, vias 5 -> 50
- net /ADC2: track 56.7 -> 61.8 mm
- net /ADC3: track 47.4 -> 51.1 mm
- net (no net): vias 52 -> 1
Other:
- board text added: "BEIA T4ME2"
- board text added: "V1"

Commit message: f
Routing:
- removed copper zone on In2.Cu, net GND
Other:
- copper layers 4 -> 2
- net class Default removed
