File: toilet4me2_V2/shiled_v2/shiled_v2.kicad_sch (KiCad schematic)
At the start: 41 parts, among them J1 40HAT, J2 MOTOR, J3 Conn_01x01, J4 Conn_01x01, J5 Conn_01x01, U3 DHT11, U4 CAT24C32-raspberrypi_hat

Commit message: g
Parts:
- removed J2: MOTOR, Connector_PinHeader_2.54mm:PinHeader_1x02_P2.54mm_Vertical, symbol Connector:Conn_01x02_Male
- added C10, C8: 1u, Capacitor_SMD:C_0805_2012Metric_Pad1.18x1.45mm_HandSolder, symbol Device:C_Small
- added C7: 100n, Capacitor_SMD:C_0805_2012Metric_Pad1.18x1.45mm_HandSolder, symbol Device:C_Small
- added D2: (no value), symbol Device:D_Small
- added D3: D_Small, Diode_SMD:D_SOD-123, symbol Device:D_Small
- added J2, J5: (no value), symbol Connector_Generic:Conn_01x03
- added J?: Conn_01x01, Connector_PinHeader_2.54mm:PinHeader_1x01_P2.54mm_Vertical, symbol Connector_Generic:Conn_01x01
- added L1: (no value), symbol Device:L_Small
- added R10, R11, R12: (no value), Resistor_SMD:R_0805_2012Metric_Pad1.20x1.40mm_HandSolder, symbol Device:R_Small
- added R17, R18, R7: 5k1, Resistor_SMD:R_0805_2012Metric_Pad1.20x1.40mm_HandSolder, symbol Device:R_Small
- added R19, R20: (no value), symbol Device:R_Small
- added S1: (no value), symbol SamacSys_Parts:PTS526_SM15_SMTR2_LFS
- added U3: (no value), Package_TO_SOT_SMD:SOT-23-5_HandSoldering, symbol My_custom_lib:AP3012KTR-G1
- added U7: (no value), symbol My_custom_lib:MCP47DA1
- C5: value (none) -> 100n; footprint (none) -> Capacitor_SMD:C_0805_2012Metric_Pad1.18x1.45mm_HandSolder
- C6: value (none) -> 1u; footprint (none) -> Capacitor_SMD:C_0805_2012Metric_Pad1.18x1.45mm_HandSolder
- C9: renamed from C7; value (none) -> 1u; footprint (none) -> Capacitor_SMD:C_0805_2012Metric_Pad1.18x1.45mm_HandSolder
- D1: value (none) -> D_Small; footprint (none) -> Diode_SMD:D_SOD-123
- FID1: value Fiducial -> (none); footprint Fiducial:Fiducial_1.5mm_Mask3mm -> (none); now left out of the parts list
- FID2: now left out of the parts list
- H1, H2, H3, H4: value 3mm_Mounting_Hole -> (none); footprint project_footprints:NPTH_3mm_ID -> (none); now left out of the parts list
- Q1: value (none) -> Q_NMOS_DGS; footprint (none) -> Package_TO_SOT_THT:TO-92_HandSolder
- R13: renamed from R9; value (none) -> 3K9; footprint (none) -> Resistor_SMD:R_0805_2012Metric_Pad1.20x1.40mm_HandSolder
- R4: value (none) -> 1k-100
- R5: value 220+ -> (none); footprint Resistor_THT:R_Axial_DIN0204_L3.6mm_D1.6mm_P7.62mm_Horizontal -> (none)
- R6: value 10k -> (none); footprint Resistor_THT:R_Axial_DIN0204_L3.6mm_D1.6mm_P7.62mm_Horizontal -> (none)
- R8: renamed from R7; value (none) -> 5k1
- RV1: value (none) -> 100k; footprint (none) -> Potentiometer_THT:Potentiometer_Piher_PT-10-V05_Vertical
- U1: value (none) -> LM4040DBZ-4.1; footprint (none) -> Package_TO_SOT_SMD:SOT-23
- U2: value (none) -> MCP3208; footprint (none) -> Package_SO:SOIC-16_3.9x9.9mm_P1.27mm
- U6: renamed from U5; value (none) -> MQ-135; footprint (none) -> Sensor:MQ-6
- U8: renamed from U6; value (none) -> MQ-136
- U9: renamed from U7; value (none) -> MQ-137
- renumbered J5 to J6, R10 to R14, R8 to R9, U3 to U4, U4 to U5
Connections:
- net +3V3: now also J1.17 (P3V3), R17.2, R18.1
- net +5V: now also C8.2, J2.3 (Pin_3), L1.1, R19.2, U3.5 (Vin)
- net ADC1: now also J3.1 (Pin_1)
- net ADC2: now also J4.1 (Pin_1)
- net ADC3: now also J6.1 (Pin_1)
- net DHT11: now also J1.15 (BCM22); no longer J1.10 (BCM15)
- net ENABLE: now also J1.37 (BCM26); no longer J1.16 (BCM23)
- net GND: now also C10.1, C7.1, C8.1, D3.2 (A), J5.2 (Pin_2), J?.1 (Pin_1), R11.2, R20.1, U3.2 (GND), U7.2 (Vss)
- net SDA: now reaches J1.3 (BCM2)
- net SDA: now also U7.4 (SDA)
- net SCL: now reaches J1.5 (BCM3)
- net SCL: now also U7.3 (SCL)
- net write_protect: now reaches JP1.2 (B), R9.2, U5.7 (WP)
- net nmos_gate: now reaches Q1.2 (G), R5.2, R6.1
- net at RV3.3: no longer J6.1 (Pin_1)
- net at D1.2 (A), Q1.1 (D): now also J2.2 (Pin_2)
- net at RV1.3: no longer J3.1 (Pin_1)
- net at RV2.3: no longer J4.1 (Pin_1)
- new net: R7.2, S1.1 (COM_1), S1.2 (COM_2)
- new net +12V: C10.2, D2.1 (K), D3.1 (K), J5.3 (Pin_3), R10.1
- new net DAC_out: R12.2, U7.5 (VOut)
- new net FB_pin: R10.2, R11.1, R12.1, U3.3 (FB)
- new net RST: C7.2, S1.3 (NO_1), S1.4 (NO_2)
- new net SW_node: D2.2 (A), L1.2, U3.1 (SW)
- new net quasi_3v3: R19.1, R20.2, R7.1
- new net tact: J2.1 (Pin_1), R17.1
- new net tact2: J5.1 (Pin_1), R18.2
- no-connect marks 5 -> 8
Other:
- note added: "1k8 pull ups to 3V3 allready built in"
- note added: "Soft Reset"
- note added: "active high"
- note added: "pull ups"
- note added: "quasi 3v3"
- moved on the sheet: J3, J4, J6, RV3
