File: toilet4me2_V2/shiled_v2/shiled_v2.kicad_sch (KiCad schematic)
At the start: 68 parts, among them J1 40HAT, J2 Motor1, J3 Conn_01x01, J4 Conn_01x01, J5 Motor2, J6 Conn_01x01, J7 Conn_01x01, Q1 Q_NMOS_DGS, U1 LM4040DBZ-4.1, U2 MCP3208, U3 AP3012KTR-G1, U4 DHT11, U5 CAT24C32-raspberrypi_hat, U6 MQ-135, U7 MCP47DA1, U8 MQ-136, U9 MQ-137

Commit message: Update shiled_v2.kicad_sch
Parts:
- R10: value 91k -> 100k
- R11: value 10k -> 5k6
- R12: value 18k -> 5k6
- R16, R17, R18: value 5k1 -> 5k6
Other:
- note added: "1/6.6 voltage divider so 26V max on this pin"
Changed lines of the file:
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@@
     (effects (font (size 1 1)) (justify left bottom))
+  )
+  (text "1/6.6 voltage divider\nso 26V max on this pin" (at 227.965 130.81 0)
+    (effects (font (size 1.27 1.27)) (justify left bottom))
   )
   (text "MOTOR CONTROL OLD" (at 108.585 223.52 0)
@@
       (effects (font (size 1.27 1.27)) (justify left))
     )
-    (property "Value" "10k" (id 1) (at 177.165 174.625 0)
+    (property "Value" "5k6" (id 1) (at 177.165 174.625 0)
       (effects (font (size 1.27 1.27)) (justify left))
     )
@@
       (effects (font (size 1.27 1.27)) (justify left))
     )
-    (property "Value" "91k" (id 1) (at 177.165 159.7914 0)
+    (property "Value" "100k" (id 1) (at 177.165 159.7914 0)
       (effects (font (size 1.27 1.27)) (justify left))
     )
@@
       (effects (font (size 1.27 1.27)) (justify left))
     )
-    (property "Value" "18k" (id 1) (at 186.3725 167.5511 90)
+    (property "Value" "5k6" (id 1) (at 186.3725 167.5511 90)
       (effects (font (size 1.27 1.27)) (justify left))
     )
@@
       (effects (font (size 1.27 1.27)) (justify left))
     )
-    (property "Value" "5k1" (id 1) (at 257.81 133.35 0)
+    (property "Value" "5k6" (id 1) (at 257.81 133.35 0)
       (effects (font (size 1.27 1.27)) (justify left))
     )
@@
       (effects (font (size 1.27 1.27)) (justify left))
     )
-    (property "Value" "5k1" (id 1) (at 289.56 136.1186 0)
+    (property "Value" "5k6" (id 1) (at 289.56 136.1186 0)
       (effects (font (size 1.27 1.27)) (justify left))
     )
@@
       (effects (font (size 1.27 1.27)) (justify left))
     )
-    (property "Value" "5k1" (id 1) (at 283.21 135.89 0)
+    (property "Value" "5k6" (id 1) (at 283.21 135.89 0)
       (effects (font (size 1.27 1.27)) (justify left))
     )
@@
     )
     (path "/23074297-972e-4551-8f73-ec0134c4aadf"
-      (reference "R10") (unit 1) (value "91k") (footprint "Resistor_SMD:R_0805_2012Metric_Pad1.20x1.40mm_HandSolder")
+      (reference "R10") (unit 1) (value "100k") (footprint "Resistor_SMD:R_0805_2012Metric_Pad1.20x1.40mm_HandSolder")
     )
     (path "/19e1d4d7-79f8-471d-82eb-d45439823a9c"
-      (reference "R11") (unit 1) (value "10k") (footprint "Resistor_SMD:R_0805_2012Metric_Pad1.20x1.40mm_HandSolder")
+      (reference "R11") (unit 1) (value "5k6") (footprint "Resistor_SMD:R_0805_2012Metric_Pad1.20x1.40mm_HandSolder")
     )
     (path "/9dc3232e-1f61-4d94-ad2c-bb3e9e9f0416"
-      (reference "R12") (unit 1) (value "18k") (footprint "Resistor_SMD:R_0805_2012Metric_Pad1.20x1.40mm_HandSolder")
+      (reference "R12") (unit 1) (value "5k6") (footprint "Resistor_SMD:R_0805_2012Metric_Pad1.20x1.40mm_HandSolder")
     )
     (path "/352e772a-2599-4a55-81ac-32c8c70c5cb0"
@@
     )
     (path "/a8542623-53bd-4b45-8dfa-a8734b194b4c"
-      (reference "R16") (unit 1) (value "5k1") (footprint "Resistor_SMD:R_0805_2012Metric_Pad1.20x1.40mm_HandSolder")
+      (reference "R16") (unit 1) (value "5k6") (footprint "Resistor_SMD:R_0805_2012Metric_Pad1.20x1.40mm_HandSolder")
     )
     (path "/dc88d5f9-a711-458e-9321-0d7ef5df941d"
-      (reference "R17") (unit 1) (value "5k1") (footprint "Resistor_SMD:R_0805_2012Metric_Pad1.20x1.40mm_HandSolder")
+      (reference "R17") (unit 1) (value "5k6") (footprint "Resistor_SMD:R_0805_2012Metric_Pad1.20x1.40mm_HandSolder")
     )
     (path "/d030de14-58e3-424d-980c-ddea037cfeed"
-      (reference "R18") (unit 1) (value "5k1") (footprint "Resistor_SMD:R_0805_2012Metric_Pad1.20x1.40mm_HandSolder")
+      (reference "R18") (unit 1) (value "5k6") (footprint "Resistor_SMD:R_0805_2012Metric_Pad1.20x1.40mm_HandSolder")
     )
     (path "/8251a3f3-2c5c-4c20-aeb6-e0a9b4fd81b4"

Commit message: f
Parts:
- R11, R12: value 5k6 -> 10k
Changed lines of the file:
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@@
     (effects (font (size 1.27 1.27)) (justify left bottom))
   )
-  (text "hysteresis:\nhigh:0.7Vdd\nlow :0.3Vdd" (at 190.5 189.865 0)
+  (text "hysteresis:\nhigh:0.7Vdd\nlow :0.3Vdd" (at 226.695 185.42 0)
     (effects (font (size 1 1)) (justify left bottom))
   )
@@
   )
   (text "poate trebuie pussa o dioda pe alimenare\npt a redice Vdd la 3.3/0.7  sau mai putin\n(4.71V)"
-    (at 202.565 190.5 0)
+    (at 238.76 186.055 0)
     (effects (font (size 1 1)) (justify left bottom))
   )
@@
     )
   )
-  (global_label "SCL" (shape input) (at 50.8 64.135 180) (fields_autoplaced)
+  (global_label "SCL" (shape bidirectional) (at 50.8 64.135 180) (fields_autoplaced)
     (effects (font (size 1.27 1.27)) (justify right))
-    (property "Intersheet References" "${INTERSHEET_REFS}" (id 0) (at 44.6888 64.2144 0)
+    (property "Intersheet References" "${INTERSHEET_REFS}" (id 0) (at 44.6888 64.0556 0)
       (effects (font (size 1.27 1.27)) (justify right) hide)
     )
@@
     )
   )
-  (global_label "SDA" (shape input) (at 50.8 61.595 180) (fields_autoplaced)
+  (global_label "SDA" (shape bidirectional) (at 50.8 61.595 180) (fields_autoplaced)
     (effects (font (size 1.27 1.27)) (justify right))
-    (property "Intersheet References" "${INTERSHEET_REFS}" (id 0) (at 44.6283 61.6744 0)
+    (property "Intersheet References" "${INTERSHEET_REFS}" (id 0) (at 44.6283 61.5156 0)
       (effects (font (size 1.27 1.27)) (justify right) hide)
     )
@@
       (effects (font (size 1.27 1.27)) (justify left))
     )
-    (property "Value" "5k6" (id 1) (at 177.165 174.625 0)
+    (property "Value" "10k" (id 1) (at 177.165 174.625 0)
       (effects (font (size 1.27 1.27)) (justify left))
     )
@@
       (effects (font (size 1.27 1.27)) (justify left))
     )
-    (property "Value" "5k6" (id 1) (at 186.3725 167.5511 90)
+    (property "Value" "10k" (id 1) (at 186.3725 167.5511 90)
       (effects (font (size 1.27 1.27)) (justify left))
     )
@@
     )
     (path "/19e1d4d7-79f8-471d-82eb-d45439823a9c"
-      (reference "R11") (unit 1) (value "5k6") (footprint "Resistor_SMD:R_0805_2012Metric_Pad1.20x1.40mm_HandSolder")
+      (reference "R11") (unit 1) (value "10k") (footprint "Resistor_SMD:R_0805_2012Metric_Pad1.20x1.40mm_HandSolder")
     )
     (path "/9dc3232e-1f61-4d94-ad2c-bb3e9e9f0416"
-      (reference "R12") (unit 1) (value "5k6") (footprint "Resistor_SMD:R_0805_2012Metric_Pad1.20x1.40mm_HandSolder")
+      (reference "R12") (unit 1) (value "10k") (footprint "Resistor_SMD:R_0805_2012Metric_Pad1.20x1.40mm_HandSolder")
     )
     (path "/352e772a-2599-4a55-81ac-32c8c70c5cb0"

Commit message: t
Parts:
- added C12: 1u, Capacitor_SMD:C_0805_2012Metric_Pad1.18x1.45mm_HandSolder, symbol Device:C_Small
- added JP2: addres, Jumper:SolderJumper-3_P1.3mm_Bridged12_Pad1.0x1.5mm, symbol Jumper:Jumper_3_Bridged12
- added U10: BME280/BME680, Package_LGA:Bosch_LGA-8_2.5x2.5mm_P0.65mm_ClockwisePinNumbering, symbol Sensor:BME280
Connections:
- net +3V3: now also C12.2, JP2.3 (B), U10.2 (CSB), U10.6 (VDDIO), U10.8 (VDD)
- net GND: now also C12.1, JP2.1 (A), U10.1 (GND), U10.7 (GND)
- net SCL: now also U10.4 (SCK)
- net SDA: now also U10.3 (SDI)
- new net: JP2.2 (C), U10.5 (SDO)
Other:
- note added: "LSD adress: GND -> 0 VCC -> 1"
