File: toilet4me2_V2/shiled_v2/shiled_v2.kicad_pcb (KiCad board)
At the start: 2 copper layers, 65 x 56 mm, 40 parts, among them J1 40HAT, J2 MOTOR, J3 Conn_01x01, J4 Conn_01x01, J5 Conn_01x01, Q1 Q_NMOS_DGS, U1 LM4040DBZ-4.1, U2 MCP3208, U3 DHT11, U4 CAT24C32-raspberrypi_hat, U5 MQ-135, U6 MQ-136, U7 MQ-137

Commit message: g
Parts:
- added C10: 1u, Capacitor_SMD:C_0805_2012Metric_Pad1.18x1.45mm_HandSolder, F.Cu at (92.8, 77.1)
- added C7: 100n, Capacitor_SMD:C_0805_2012Metric_Pad1.18x1.45mm_HandSolder, F.Cu at (95.0, 112.3)
- added C8: 1u, Capacitor_SMD:C_0805_2012Metric_Pad1.18x1.45mm_HandSolder, F.Cu at (94.6, 68.8)
- added D1: D_Small, Diode_SMD:D_SOD-123, F.Cu at (84.6, 82.2)
- added D2: D_Small, Diode_SMD:D_SOD-123, F.Cu at (90.4, 76.1)
- added D3: D_Small, Diode_SMD:D_SOD-123, F.Cu at (85.1, 73.8)
- added J5: Motor2, Connector_PinHeader_2.54mm:PinHeader_1x03_P2.54mm_Vertical, F.Cu at (81.3, 70.1)
- added L1: L_Small, Inductor_SMD:L_Taiyo-Yuden_MD-5050, F.Cu at (89.5, 70.7)
- added R10: 91k, Resistor_SMD:R_0805_2012Metric_Pad1.20x1.40mm_HandSolder, F.Cu at (96.0, 78.2)
- added R11: 10k, Resistor_SMD:R_0805_2012Metric_Pad1.20x1.40mm_HandSolder, F.Cu at (96.0, 76.1)
- added R12: 18k, Resistor_SMD:R_0805_2012Metric_Pad1.20x1.40mm_HandSolder, F.Cu at (99.4, 77.2)
- added R17: 5k1, Resistor_SMD:R_0805_2012Metric_Pad1.20x1.40mm_HandSolder, F.Cu at (105.0, 83.4)
- added R18: 5k1, Resistor_SMD:R_0805_2012Metric_Pad1.20x1.40mm_HandSolder, F.Cu at (109.1, 83.4)
- added R19: 10k, Resistor_SMD:R_0805_2012Metric_Pad1.20x1.40mm_HandSolder, F.Cu at (81.3, 106.0)
- added R20: 20k, Resistor_SMD:R_0805_2012Metric_Pad1.20x1.40mm_HandSolder, F.Cu at (81.3, 108.1)
- added R7: 5k1, Resistor_SMD:R_0805_2012Metric_Pad1.20x1.40mm_HandSolder, F.Cu at (84.2, 107.5)
- added S1: PTS526_SM15_SMTR2_LFS, SamacSys_Parts:PTS526SM15SMTR2LFS, F.Cu at (89.5, 108.9)
- added U3: AP3012KTR-G1, Package_TO_SOT_SMD:SOT-23-5_HandSoldering, F.Cu at (94.5, 72.5)
- added U7: MCP47DA1, Package_TO_SOT_SMD:SOT-23-6_Handsoldering, F.Cu at (99.4, 72.4)
- added kibuzzard-62DA5EB2: G***, kibuzzard-62DA5EB2, F.Cu at (140.7, 105.2)
- FID2: moved to B.Cu
- J2: value MOTOR -> Motor1; footprint Connector_PinHeader_2.54mm:PinHeader_1x02_P2.54mm_Vertical -> Connector_PinHeader_2.54mm:PinHeader_1x03_P2.54mm_Vertical
- R5, R6: footprint Resistor_THT:R_Axial_DIN0204_L3.6mm_D1.6mm_P7.62mm_Horizontal -> Resistor_THT:R_Axial_DIN0204_L3.6mm_D1.6mm_P2.54mm_Vertical
- moved J2 134.7 mm to (81.3, 79.4)
- moved Q1 117.9 mm to (88.1, 80.9), turned to -90 degrees
- moved R5 100.6 mm to (94.9, 82.1), turned to -90 degrees
- moved JP1 99.8 mm to (123.5, 76.3), turned to -90 degrees
- moved R8 97.3 mm to (105.7, 73.5), turned to 0 degrees
- moved U4 94.4 mm to (104.7, 78.0), turned to 90 degrees
- moved R6 86.7 mm to (98.2, 83.9)
- moved R2 55.0 mm to (126.6, 82.8), turned to 180 degrees
- moved FID2 53.3 mm to (141.0, 104.1), turned to 180 degrees
- moved C2 52.7 mm to (126.6, 80.7), turned to 180 degrees
- moved R1 49.7 mm to (121.2, 80.1), turned to -90 degrees
- moved C1 48.2 mm to (123.4, 80.2), turned to -90 degrees
- moved R3 46.9 mm to (133.5, 82.9), turned to -90 degrees
- moved C3 43.7 mm to (135.6, 82.9), turned to 90 degrees
- moved J6 15.3 mm to (123.3, 112.1)
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- renumbered C7 to C9, J5 to J6, R9 to R13, R10 to R14, R7 to R8, R8 to R9, U3 to U4, U4 to U5, U5 to U6, U6 to U8, U7 to U9
Connections:
- net Net-(JP1-Pad2) renamed /write_protect
- net Net-(Q1-Pad2) renamed /nmos_gate
- J1 pad 10: /DHT11 -> unconnected-(J1-Pad10)
- J1 pad 15: unconnected-(J1-Pad15) -> /DHT11
- J1 pad 16: /ENABLE -> unconnected-(J1-Pad16)
- J1 pad 17: unconnected-(J1-Pad17) -> +3V3
- J1 pad 3: unconnected-(J1-Pad3) -> SDA
- J1 pad 37: unconnected-(J1-Pad37) -> /ENABLE
- J1 pad 5: unconnected-(J1-Pad5) -> SCL
- J2 pad 1: +5V -> tact
- J3 pad 1: Net-(J3-Pad1) -> /ADC1
- J4 pad 1: Net-(J4-Pad1) -> /ADC2
- J6 pad 1: Net-(J5-Pad1) -> /ADC3
- RV1 pad 3: Net-(J3-Pad1) -> unconnected-(RV1-Pad3)
- RV2 pad 3: Net-(J4-Pad1) -> unconnected-(RV2-Pad3)
- RV3 pad 3: Net-(J5-Pad1) -> unconnected-(RV3-Pad3)
Routing:
- net +5V: track 0.00 -> 219.5 mm, vias 0 -> 8
- net GND: track 0.00 -> 60.1 mm, vias 0 -> 30
- net /ADC1: track 0.00 -> 56.6 mm
- net +3V3: track 0.00 -> 47.6 mm, vias 0 -> 2
- net /ADC2: track 0.00 -> 42.1 mm
- net tact2: track 0.00 -> 38.2 mm, vias 0 -> 1
- net /ADC3: track 0.00 -> 33.9 mm
- net /motor_control1: track 0.00 -> 26.1 mm, vias 0 -> 4
- net tact: track 0.00 -> 25.6 mm
- net SDA: track 0.00 -> 15.2 mm
- net +12V: track 0.00 -> 15.0 mm
- net /DHT11: track 0.00 -> 13.4 mm
- net /ENABLE: track 0.00 -> 13.3 mm, vias 0 -> 1
- net /DIN: track 0.00 -> 12.8 mm
- net /CLK: track 0.00 -> 12.2 mm, vias 0 -> 2
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- added copper zone on F.Cu, net +12V
- added copper zone on F.Cu, net +5V
- added copper zone on F.Cu, net /SW_node
- added copper zone on F.Cu, net GND

Commit message: k
Parts:
- added C11: 100n, Capacitor_SMD:C_0805_2012Metric_Pad1.18x1.45mm_HandSolder, F.Cu at (101.2, 68.7)
- added CH4: -, TestPoint:TestPoint_THTPad_D1.0mm_Drill0.5mm, F.Cu at (142.0, 73.4)
- added CH5: -, TestPoint:TestPoint_THTPad_D1.0mm_Drill0.5mm, F.Cu at (137.8, 81.7)
- added CH6: -, TestPoint:TestPoint_THTPad_D1.0mm_Drill0.5mm, F.Cu at (142.1, 76.9)
- added CH7: -, TestPoint:TestPoint_THTPad_D1.0mm_Drill0.5mm, F.Cu at (142.0, 79.2)
- added J7: Conn_01x01, Connector_PinHeader_2.54mm:PinHeader_1x01_P2.54mm_Vertical, F.Cu at (94.6, 114.0)
- added R15: 10K, Resistor_SMD:R_0805_2012Metric_Pad1.20x1.40mm_HandSolder, F.Cu at (97.5, 70.5)
- added R16: 5k1, Resistor_SMD:R_0805_2012Metric_Pad1.20x1.40mm_HandSolder, F.Cu at (117.6, 84.8)
- added R21: 1k, Resistor_SMD:R_0805_2012Metric_Pad1.20x1.40mm_HandSolder, F.Cu at (117.6, 82.7)
- added kibuzzard-62E789B0: G***, kibuzzard-62E789B0, F.Cu at (141.8, 89.5)
- added kibuzzard-62E797EE: G***, kibuzzard-62E797EE, F.Cu at (89.2, 101.7)
- added kibuzzard-62E797F8: G***, kibuzzard-62E797F8, F.Cu at (109.2, 101.9)
- added kibuzzard-62E79804: G***, kibuzzard-62E79804, F.Cu at (130.0, 101.9)
- added kibuzzard-62E79C6C: G***, kibuzzard-62E79C6C, F.Cu at (108.5, 79.9)
- added kibuzzard-62E79CA0: G***, kibuzzard-62E79CA0, F.Cu at (110.4, 74.0)
- L1: value L_Small -> 10uH
- R1, R2, R3: value 1k-100 -> 1k
- moved C7 63.2 mm to (141.2, 69.2), turned to 0 degrees
- moved FID2 2.34 mm to (140.1, 106.3)
- moved U7 1.56 mm to (101.0, 72.2)
- moved R17 0.61 mm to (105.0, 82.8)
- moved R18 0.59 mm to (108.9, 82.8)
- moved S1 0.50 mm to (89.2, 108.6)
- moved RV1 0.49 mm to (101.1, 108.2)
- moved U9 0.45 mm to (133.4, 98.6)
- moved C3 0.38 mm to (135.3, 82.9)
- moved R3 0.33 mm to (133.2, 82.9)
- moved C8 0.30 mm to (94.3, 68.9)
- moved R7 0.26 mm to (84.0, 107.3)
- moved R19 0.23 mm to (81.0, 106.0)
- moved R20 0.23 mm to (81.0, 108.1)
Connections:
- net /Vref renamed /Vref_4.096V
- net Net-(D1-Pad2) renamed /old_fan_low_side
- J1 pad 11: unconnected-(J1-Pad11) -> /BOOST_ENABLE
- J1 pad 36: unconnected-(J1-Pad36) -> RST
- R7 pad 2: Net-(R7-Pad2) -> RST
- S1 pad 1: Net-(R7-Pad2) -> RST
- S1 pad 2: Net-(R7-Pad2) -> RST
- S1 pad 3: RST -> GND
- S1 pad 4: RST -> GND
- U2 pad 4: unconnected-(U2-Pad4) -> /12V_sense
- U2 pad 5: unconnected-(U2-Pad5) -> Net-(CH4-Pad1)
- U2 pad 6: unconnected-(U2-Pad6) -> Net-(CH5-Pad1)
- U2 pad 7: unconnected-(U2-Pad7) -> Net-(CH6-Pad1)
- U2 pad 8: unconnected-(U2-Pad8) -> Net-(CH7-Pad1)
- U3 pad 4: unconnected-(U3-Pad4) -> /BOOST_ENABLE
- U7 pad 1: unconnected-(U7-Pad1) -> +3V3
- U7 pad 6: unconnected-(U7-Pad6) -> +3V3
Routing:
- net RST: track 8.64 -> 123.1 mm
- net +12V: track 15.0 -> 39.6 mm, vias 0 -> 2
- net /12V_sense: track 0.00 -> 24.0 mm
- net GND: track 60.1 -> 83.7 mm, vias 30 -> 50
- net +3V3: track 47.6 -> 60.7 mm, vias 2 -> 5
- net /BOOST_ENABLE: track 0.00 -> 9.73 mm, vias 0 -> 1
- net Net-(CH4-Pad1): track 0.00 -> 9.71 mm
- net Net-(R7-Pad2): track 8.57 -> 0.00 mm
- net Net-(CH6-Pad1): track 0.00 -> 4.94 mm
- net Net-(CH5-Pad1): track 0.00 -> 3.02 mm
- net /ADC1: track 56.6 -> 59.0 mm
- net /motor_control1: track 26.1 -> 28.4 mm, vias 4 -> 2
- net Net-(CH7-Pad1): track 0.00 -> 2.17 mm
- net SDA: track 15.2 -> 16.6 mm
- net SCL: track 10.3 -> 11.7 mm
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Other:
- board text added: "12V"
- board text added: "5V"
- board text added: "D"
- board text added: "G"
- board text added: "GND"
- board text added: "S"
- board text added: "TACT1"
- board text added: "TACT2"

Commit message: v1
Parts:
- added kibuzzard-62EB9840: G***, kibuzzard-62EB9840, F.Cu at (139.0, 85.9)
Changed lines of the file:
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@@
     (pad "6" thru_hole circle (at 6.72 0 90) (size 2 2) (drill 1) (layers *.Cu *.Mask)
       (net 3 "+5V") (pinfunction "A1") (pintype "passive"))
-    (model "F:/MQ_sensor_3D_model_B-Body.wrl"
+    (model "C:/Users/robert_alfred.kecs/Documents/KiCad/my_3D_models/MQ_sensor_3D_model_B-Body.wrl"
       (offset (xyz 3.5 -3.25 2))
       (scale (xyz 0.4 0.4 0.4))
@@
     (property "Sheetname" "")
     (attr smd)
-    (fp_text reference "C3" (at -1.0414 1.905 180) (layer "F.SilkS")
+    (fp_text reference "C3" (at -2.6162 0.1016 180) (layer "F.SilkS")
       (effects (font (size 1 1) (thickness 0.15)))
     )
@@
     (pad "6" thru_hole circle (at 6.72 0 90) (size 2 2) (drill 1) (layers *.Cu *.Mask)
       (net 3 "+5V") (pinfunction "A1") (pintype "passive"))
-    (model "F:/MQ_sensor_3D_model_B-Body.wrl"
+    (model "C:/Users/robert_alfred.kecs/Documents/KiCad/my_3D_models/MQ_sensor_3D_model_B-Body.wrl"
       (offset (xyz 3.5 -3.25 2))
       (scale (xyz 0.4 0.4 0.4))
@@
       (rotate (xyz 0 0 0))
     )
+  )
+  (footprint "kibuzzard-62EB9840" (layer "F.Cu")
+    (at 139.0396 85.9028 90)
+    (descr "Converted using: scripting")
+    (tags "svg2mod")
+    (attr board_only exclude_from_pos_files exclude_from_bom)
+    (fp_text reference "kibuzzard-62EB9840" (at 0 -1.042305 90) (layer "F.SilkS") hide
+      (effects (font (size 0.000254 0.000254) (thickness 0.000003)))
+    )
+    (fp_text value "G***" (at 0 1.042305 90) (layer "F.SilkS") hide
+      (effects (font (size 0.000254 0.000254) (thickness 0.000003)))
+    )
+    (fp_poly (pts
+        (xy -2.271713 -1.041797)
+        (xy -2.271713 -0.869156)
+        (xy -1.997869 -0.869156)
+        (xy -1.726406 0.631031)
+        (xy -1.724025 0.631031)
+        (xy -1.452563 -0.869156)
+        (xy -1.188244 -0.869156)
+        (xy -0.802481 -0.815578)
+        (xy -0.686395 -0.873621)
+        (xy -0.538163 -0.892969)
+        (xy -0.38993 -0.873621)
+        (xy -0.273844 -0.815578)
+        (xy -0.184845 -0.707827)
+        (xy -0.117872 -0.539353)
+        (xy -0.086783 -0.391054)
+        (xy -0.06813 -0.21127)
+        (xy -0.061913 0)
+        (xy -0.06813 0.21127)
+        (xy -0.086783 0.391054)
+        (xy -0.117872 0.539353)
+        (xy -0.184845 0.707827)
+        (xy -0.273844 0.815578)
+        (xy -0.38993 0.873621)
+        (xy -0.538163 0.892969)
+        (xy -0.686395 0.873621)
+        (xy -0.802481 0.815578)
+        (xy -0.89148 0.707827)
+        (xy -0.958453 0.539353)
+        (xy -0.989542 0.391054)
+        (xy -1.008195 0.21127)
+        (xy -1.014412 0)
+        (xy -1.008195 -0.21127)
+        (xy -0.989542 -0.391054)
+        (xy -0.958453 -0.539353)
+        (xy -0.89148 -0.707827)
+        (xy -0.802481 -0.815578)
+        (xy -1.188244 -0.869156)
+        (xy -1.576388 0.869156)
+        (xy -1.88595 0.869156)
+        (xy -2.271713 -0.869156)
+        (xy -2.271713 -1.041797)
+        (xy -2.420541 -1.041797)
+        (xy -2.420541 1.041797)
+        (xy 0.466725 0.869156)
+        (xy 0.466725 0.464344)
+        (xy 0.847725 0.464344)
+        (xy 0.847725 0.869156)
+        (xy 0.466725 0.869156)
+        (xy -2.420541 1.041797)
+        (xy -2.271713 1.041797)
+        (xy 2.271713 1.041797)
+        (xy 2.271713 0.869156)
+        (xy 1.414463 0.869156)
+        (xy 1.414463 0.661988)
+        (xy 1.567348 0.484268)
+        (xy 1.696714 0.314422)
+        (xy 1.802558 0.152449)
+        (xy 1.884881 -0.001652)
+        (xy 1.943683 -0.14788)
+        (xy 1.978965 -0.286236)
+        (xy 1.990725 -0.416719)
+        (xy 1.977926 -0.538163)
+        (xy 1.939528 -0.621506)
+        (xy 1.783556 -0.6858)
+        (xy 1.671638 -0.67019)
+        (xy 1.548606 -0.623358)
+        (xy 1.414463 -0.545306)
+        (xy 1.414463 -0.769144)
+        (xy 1.546225 -0.837935)
+        (xy 1.687513 -0.87921)
+        (xy 1.838325 -0.892969)
+        (xy 2.019002 -0.863501)
+        (xy 2.151459 -0.775097)
+        (xy 2.23272 -0.629543)
+        (xy 2.259806 -0.428625)
+        (xy 2.244857 -0.277813)
+        (xy 2.20001 -0.117475)
+        (xy 2.125266 0.052388)
+        (xy 2.047652 0.188416)
+        (xy 1.949351 0.334566)
+        (xy 1.830363 0.490835)
+        (xy 1.690688 0.657225)
+        (xy 1.690688 0.661988)
+        (xy 2.271713 0.661988)
+        (xy 2.271713 0.869156)
+        (xy 2.271713 1.041797)
+        (xy 2.420541 1.041797)
+        (xy 2.420541 -1.041797)
+        (xy 2.271713 -1.041797)
+        (xy -2.271713 -1.041797)
+      ) (layer "F.SilkS") (width 0) (fill solid))
+    (fp_poly (pts
+        (xy -0.762 0.197644)
+        (xy -0.354806 -0.509588)
+        (xy -0.426244 -0.651272)
+        (xy -0.538163 -0.692944)
+        (xy -0.663178 -0.638175)
+        (xy -0.705148 -0.558403)
+        (xy -0.738188 -0.428625)
+        (xy -0.754063 -0.312208)
+        (xy -0.763588 -0.169333)
+        (xy -0.766763 0)
+        (xy -0.762 0.197644)
+      ) (layer "F.SilkS") (width 0) (fill solid))
+    (fp_poly (pts
+        (xy -0.731044 0.47625)
+        (xy -0.657225 0.644128)
+        (xy -0.538163 0.692944)
+        (xy -0.413147 0.638175)
+        (xy -0.371177 0.558403)
+        (xy -0.338138 0.428625)
+        (xy -0.322263 0.312208)
+        (xy -0.312738 0.169333)
+        (xy -0.309563 0)
+        (xy -0.311348 -0.129183)
+        (xy -0.316706 -0.240506)
+        (xy -0.731044 0.47625)
+      ) (layer "F.SilkS") (width 0) (fill solid))
   )
   (footprint "Resistor_SMD:R_0805_2012Metric_Pad1.20x1.40mm_HandSolder" (layer "F.Cu")
@@
     (pad "6" thru_hole circle (at 6.72 0 90) (size 2 2) (drill 1) (layers *.Cu *.Mask)
       (net 3 "+5V") (pinfunction "A1") (pintype "passive"))
-    (model "F:/MQ_sensor_3D_model_B-Body.wrl"
+    (model "C:/Users/robert_alfred.kecs/Documents/KiCad/my_3D_models/MQ_sensor_3D_model_B-Body.wrl"
       (offset (xyz 3.5 -3.25 2))
       (scale (xyz 0.4 0.4 0.4))
@@
     (attr smd)
     (fp_text reference "U3" (at -0.4826 2.4384 90) (layer "F.SilkS")
-      (effects (font (size 0.8 0.8)))
+      (effects (font (size 0.8 0.8) (thickness 0.15)))
     )
     (fp_text value "AP3012KTR-G1" (at 0 2.9 90) (layer "F.Fab")

Commit message: t
Parts:
- added C12: 1u, Capacitor_SMD:C_0805_2012Metric_Pad1.18x1.45mm_HandSolder, F.Cu at (109.7, 73.4)
- added JP2: addres, Jumper:SolderJumper-3_P1.3mm_Bridged12_Pad1.0x1.5mm, F.Cu at (107.1, 69.9)
- added U10: BME280/BME680, Package_LGA:Bosch_LGA-8_2.5x2.5mm_P0.65mm_ClockwisePinNumbering, F.Cu at (106.2, 73.1)
- R10: value 91k -> 100k
- R12: value 18k -> 10k
- R16, R17, R18: value 5k1 -> 5k6
- moved R8 13.0 mm to (113.3, 84.0), turned to 90 degrees
- moved kibuzzard-62E79CA0 12.6 mm to (100.6, 82.0)
Routing:
- net /DHT11: track 13.4 -> 26.9 mm, vias 0 -> 2
- net +3V3: track 60.7 -> 73.8 mm, vias 5 -> 6
- net GND: track 83.7 -> 96.5 mm, vias 50 -> 85
- net SCL: track 11.7 -> 18.9 mm, vias 0 -> 2
- net SDA: track 16.6 -> 23.2 mm, vias 0 -> 2
- net +5V: track 219.2 -> 215.1 mm
- net Net-(JP2-Pad2): track 0.00 -> 2.26 mm
- net +12V: track 39.6 -> 41.3 mm
- net RST: track 123.1 -> 121.6 mm
- net /write_protect: track 9.64 -> 8.67 mm
- net /ADC3_filtered: track 5.79 -> 6.35 mm
- net /ADC2: track 42.2 -> 42.7 mm
