File: irigatii2/untitled.kicad_sch (KiCad schematic)
At the start: 59 parts, among them J5 valve, J6 valve, J7 valve, J8 valve, J9 valve, Q11 PMOS, Q12 PMOS, Q13 PMOS, Q14 PMOS, Q15 NMOS, Q16 NMOS, Q17 NMOS, Q18 NMOS, Q19 NMOS, Q20 NMOS, Q21 NMOS, Q22 NMOS, Q23 PMOS, Q24 PMOS, Q25 PMOS, Q26 PMOS, Q27 NMOS, Q28 NMOS, Q29 NMOS, Q30 NMOS, Q31 NMOS, Q32 NMOS, Q33 NMOS, Q34 NMOS, Q35 PMOS, Q36 PMOS, Q37 NMOS, Q38 NMOS

Commit message: j
Parts:
- R20, R21, R22, R23, R24, R25, R26, R27, R28, R29, R30, R31, R32, R33, R35, R36, R37, R38, R39, R40: footprint Resistor_THT:R_Axial_DIN0207_L6.3mm_D2.5mm_P10.16mm_Horizontal -> Resistor_THT:R_Axial_DIN0204_L3.6mm_D1.6mm_P5.08mm_Vertical
- R34: footprint Resistor_THT:R_Axial_DIN0207_L6.3mm_D2.5mm_P10.16mm_Horizontal -> Resistor_THT:R_Axial_DIN0204_L3.6mm_D1.6mm_P5.08mm_Horizontal
Changed lines of the file:
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@@
     (property "Reference" "R40" (id 0) (at 73.025 240.665 90))
     (property "Value" "100k" (id 1) (at 73.025 243.205 90))
-    (property "Footprint" "Resistor_THT:R_Axial_DIN0207_L6.3mm_D2.5mm_P10.16mm_Horizontal" (id 2) (at 73.025 238.125 0)
+    (property "Footprint" "Resistor_THT:R_Axial_DIN0204_L3.6mm_D1.6mm_P5.08mm_Vertical" (id 2) (at 73.025 238.125 0)
       (effects (font (size 1.27 1.27)) hide)
     )
@@
     (property "Reference" "R37" (id 0) (at 152.4 150.495 90))
     (property "Value" "100k" (id 1) (at 149.86 150.495 90))
-    (property "Footprint" "Resistor_THT:R_Axial_DIN0207_L6.3mm_D2.5mm_P10.16mm_Horizontal" (id 2) (at 154.94 150.495 0)
+    (property "Footprint" "Resistor_THT:R_Axial_DIN0204_L3.6mm_D1.6mm_P5.08mm_Vertical" (id 2) (at 154.94 150.495 0)
       (effects (font (size 1.27 1.27)) hide)
     )
@@
     (property "Reference" "R22" (id 0) (at 254.635 37.465 90))
     (property "Value" "100k" (id 1) (at 252.095 37.465 90))
-    (property "Footprint" "Resistor_THT:R_Axial_DIN0207_L6.3mm_D2.5mm_P10.16mm_Horizontal" (id 2) (at 257.175 37.465 0)
+    (property "Footprint" "Resistor_THT:R_Axial_DIN0204_L3.6mm_D1.6mm_P5.08mm_Vertical" (id 2) (at 257.175 37.465 0)
       (effects (font (size 1.27 1.27)) hide)
     )
@@
     (property "Reference" "R26" (id 0) (at 33.655 71.755 90))
     (property "Value" "100k" (id 1) (at 31.115 71.755 90))
-    (property "Footprint" "Resistor_THT:R_Axial_DIN0207_L6.3mm_D2.5mm_P10.16mm_Horizontal" (id 2) (at 36.195 71.755 0)
+    (property "Footprint" "Resistor_THT:R_Axial_DIN0204_L3.6mm_D1.6mm_P5.08mm_Vertical" (id 2) (at 36.195 71.755 0)
       (effects (font (size 1.27 1.27)) hide)
     )
@@
     (property "Reference" "R28" (id 0) (at 233.045 75.565 90))
     (property "Value" "100k" (id 1) (at 230.505 75.565 90))
-    (property "Footprint" "Resistor_THT:R_Axial_DIN0207_L6.3mm_D2.5mm_P10.16mm_Horizontal" (id 2) (at 235.585 75.565 0)
+    (property "Footprint" "Resistor_THT:R_Axial_DIN0204_L3.6mm_D1.6mm_P5.08mm_Vertical" (id 2) (at 235.585 75.565 0)
       (effects (font (size 1.27 1.27)) hide)
     )
@@
     (property "Reference" "R21" (id 0) (at 130.81 34.9137 90))
     (property "Value" "100k" (id 1) (at 133.35 34.9137 90))
-    (property "Footprint" "Resistor_THT:R_Axial_DIN0207_L6.3mm_D2.5mm_P10.16mm_Horizontal" (id 2) (at 128.27 34.9137 0)
+    (property "Footprint" "Resistor_THT:R_Axial_DIN0204_L3.6mm_D1.6mm_P5.08mm_Vertical" (id 2) (at 128.27 34.9137 0)
       (effects (font (size 1.27 1.27)) hide)
     )
@@
     (property "Reference" "R25" (id 0) (at 284.48 60.96 90))
     (property "Value" "100k" (id 1) (at 284.48 63.5 90))
-    (property "Footprint" "Resistor_THT:R_Axial_DIN0207_L6.3mm_D2.5mm_P10.16mm_Horizontal" (id 2) (at 284.48 58.42 0)
+    (property "Footprint" "Resistor_THT:R_Axial_DIN0204_L3.6mm_D1.6mm_P5.08mm_Vertical" (id 2) (at 284.48 58.42 0)
       (effects (font (size 1.27 1.27)) hide)
     )
@@
     (property "Reference" "R36" (id 0) (at 35.56 150.495 90))
     (property "Value" "100k" (id 1) (at 33.02 150.495 90))
-    (property "Footprint" "Resistor_THT:R_Axial_DIN0207_L6.3mm_D2.5mm_P10.16mm_Horizontal" (id 2) (at 38.1 150.495 0)
+    (property "Footprint" "Resistor_THT:R_Axial_DIN0204_L3.6mm_D1.6mm_P5.08mm_Vertical" (id 2) (at 38.1 150.495 0)
       (effects (font (size 1.27 1.27)) hide)
     )
@@
     (property "Reference" "R31" (id 0) (at 132.715 113.6537 90))
     (property "Value" "100k" (id 1) (at 135.255 113.6537 90))
-    (property "Footprint" "Resistor_THT:R_Axial_DIN0207_L6.3mm_D2.5mm_P10.16mm_Horizontal" (id 2) (at 130.175 113.6537 0)
+    (property "Footprint" "Resistor_THT:R_Axial_DIN0204_L3.6mm_D1.6mm_P5.08mm_Vertical" (id 2) (at 130.175 113.6537 0)
       (effects (font (size 1.27 1.27)) hide)
     )
@@
     (property "Reference" "R33" (id 0) (at 332.105 117.4637 90))
     (property "Value" "100k" (id 1) (at 334.645 117.4637 90))
-    (property "Footprint" "Resistor_THT:R_Axial_DIN0207_L6.3mm_D2.5mm_P10.16mm_Horizontal" (id 2) (at 329.565 117.4637 0)
+    (property "Footprint" "Resistor_THT:R_Axial_DIN0204_L3.6mm_D1.6mm_P5.08mm_Vertical" (id 2) (at 329.565 117.4637 0)
       (effects (font (size 1.27 1.27)) hide)
     )
@@
     (property "Reference" "R39" (id 0) (at 351.79 154.305 90))
     (property "Value" "100k" (id 1) (at 349.25 154.305 90))
-    (property "Footprint" "Resistor_THT:R_Axial_DIN0207_L6.3mm_D2.5mm_P10.16mm_Horizontal" (id 2) (at 354.33 154.305 0)
+    (property "Footprint" "Resistor_THT:R_Axial_DIN0204_L3.6mm_D1.6mm_P5.08mm_Vertical" (id 2) (at 354.33 154.305 0)
       (effects (font (size 1.27 1.27)) hide)
     )
@@
     (property "Reference" "R30" (id 0) (at 57.15 112.395 90))
     (property "Value" "100k" (id 1) (at 54.61 112.395 90))
-    (property "Footprint" "Resistor_THT:R_Axial_DIN0207_L6.3mm_D2.5mm_P10.16mm_Horizontal" (id 2) (at 59.69 112.395 0)
+    (property "Footprint" "Resistor_THT:R_Axial_DIN0204_L3.6mm_D1.6mm_P5.08mm_Vertical" (id 2) (at 59.69 112.395 0)
       (effects (font (size 1.27 1.27)) hide)
     )
@@
     (property "Reference" "R32" (id 0) (at 256.54 116.205 90))
     (property "Value" "100k" (id 1) (at 254 116.205 90))
-    (property "Footprint" "Resistor_THT:R_Axial_DIN0207_L6.3mm_D2.5mm_P10.16mm_Horizontal" (id 2) (at 259.08 116.205 0)
+    (property "Footprint" "Resistor_THT:R_Axial_DIN0204_L3.6mm_D1.6mm_P5.08mm_Vertical" (id 2) (at 259.08 116.205 0)
       (effects (font (size 1.27 1.27)) hide)
     )
@@
     (property "Reference" "R29" (id 0) (at 349.885 75.565 90))
     (property "Value" "100k" (id 1) (at 347.345 75.565 90))
-    (property "Footprint" "Resistor_THT:R_Axial_DIN0207_L6.3mm_D2.5mm_P10.16mm_Horizontal" (id 2) (at 352.425 75.565 0)
+    (property "Footprint" "Resistor_THT:R_Axial_DIN0204_L3.6mm_D1.6mm_P5.08mm_Vertical" (id 2) (at 352.425 75.565 0)
       (effects (font (size 1.27 1.27)) hide)
     )
@@
     (property "Reference" "R34" (id 0) (at 86.995 135.89 90))
     (property "Value" "100k" (id 1) (at 86.995 138.43 90))
-    (property "Footprint" "Resistor_THT:R_Axial_DIN0207_L6.3mm_D2.5mm_P10.16mm_Horizontal" (id 2) (at 86.995 133.35 0)
+    (property "Footprint" "Resistor_THT:R_Axial_DIN0204_L3.6mm_D1.6mm_P5.08mm_Horizontal" (id 2) (at 86.995 133.35 0)
       (effects (font (size 1.27 1.27)) hide)
     )
@@
     (property "Reference" "R35" (id 0) (at 286.385 139.7 90))
     (property "Value" "100k" (id 1) (at 286.385 142.24 90))
-    (property "Footprint" "Resistor_THT:R_Axial_DIN0207_L6.3mm_D2.5mm_P10.16mm_Horizontal" (id 2) (at 286.385 137.16 0)
+    (property "Footprint" "Resistor_THT:R_Axial_DIN0204_L3.6mm_D1.6mm_P5.08mm_Vertical" (id 2) (at 286.385 137.16 0)
       (effects (font (size 1.27 1.27)) hide)
     )
@@
     (property "Reference" "R24" (id 0) (at 85.09 57.15 90))
     (property "Value" "100k" (id 1) (at 85.09 59.69 90))
-    (property "Footprint" "Resistor_THT:R_Axial_DIN0207_L6.3mm_D2.5mm_P10.16mm_Horizontal" (id 2) (at 85.09 54.61 0)
+    (property "Footprint" "Resistor_THT:R_Axial_DIN0204_L3.6mm_D1.6mm_P5.08mm_Vertical" (id 2) (at 85.09 54.61 0)
       (effects (font (size 1.27 1.27)) hide)
     )
@@
     (property "Reference" "R38" (id 0) (at 234.95 154.305 90))
     (property "Value" "100k" (id 1) (at 232.41 154.305 90))
-    (property "Footprint" "Resistor_THT:R_Axial_DIN0207_L6.3mm_D2.5mm_P10.16mm_Horizontal" (id 2) (at 237.49 154.305 0)
+    (property "Footprint" "Resistor_THT:R_Axial_DIN0204_L3.6mm_D1.6mm_P5.08mm_Vertical" (id 2) (at 237.49 154.305 0)
       (effects (font (size 1.27 1.27)) hide)
     )
@@
     (property "Reference" "R27" (id 0) (at 150.495 71.755 90))
     (property "Value" "100k" (id 1) (at 147.955 71.755 90))
-    (property "Footprint" "Resistor_THT:R_Axial_DIN0207_L6.3mm_D2.5mm_P10.16mm_Horizontal" (id 2) (at 153.035 71.755 0)
+    (property "Footprint" "Resistor_THT:R_Axial_DIN0204_L3.6mm_D1.6mm_P5.08mm_Vertical" (id 2) (at 153.035 71.755 0)
       (effects (font (size 1.27 1.27)) hide)
     )
@@
     (property "Reference" "R20" (id 0) (at 55.245 33.655 90))
     (property "Value" "100k" (id 1) (at 52.705 33.655 90))
-    (property "Footprint" "Resistor_THT:R_Axial_DIN0207_L6.3mm_D2.5mm_P10.16mm_Horizontal" (id 2) (at 57.785 33.655 0)
+    (property "Footprint" "Resistor_THT:R_Axial_DIN0204_L3.6mm_D1.6mm_P5.08mm_Vertical" (id 2) (at 57.785 33.655 0)
       (effects (font (size 1.27 1.27)) hide)
     )
@@
     (property "Reference" "R23" (id 0) (at 330.2 38.7237 90))
     (property "Value" "100k" (id 1) (at 332.74 38.7237 90))
-    (property "Footprint" "Resistor_THT:R_Axial_DIN0207_L6.3mm_D2.5mm_P10.16mm_Horizontal" (id 2) (at 327.66 38.7237 0)
-      (effects (font (size 1.27 1.27)) hide)
-    )
+    (property "Footprint" "Resistor_THT:R_Axial_DIN0204_L3.6mm_D1.6mm_P5.08mm_Vertical" (id 2) (at 327.66 38.7237 0)
+      (effects (font (size 1.27 1.27)) hide)
+    )

Commit message: d
Connections:
- net D1_1: now also Q21.1 (G), R28.2; no longer Q19.1 (G), R26.2
- net D1_2: now also Q22.1 (G), R29.2; no longer Q20.1 (G), R27.2
- net D4_1: now also Q33.1 (G), R38.2; no longer Q21.1 (G), R28.2
- net D4_2: now also Q34.1 (G), R39.2; no longer Q22.1 (G), R29.2
- net D5_1: now also Q20.1 (G), R27.2; no longer Q33.1 (G), R38.2
- net D5_2: now also Q19.1 (G), R26.2; no longer Q34.1 (G), R39.2
Changed lines of the file:
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@@
     (effects (font (size 6 6)) (justify left bottom))
   )
-  (global_label "D1_2" (shape input) (at 166.37 67.31 0) (fields_autoplaced)
+  (global_label "D1_2" (shape input) (at 365.76 71.12 0) (fields_autoplaced)
     (effects (font (size 1.27 1.27)) (justify left))
-    (property "Intersheet References" "${INTERSHEET_REFS}" (id 0) (at 173.4398 67.3894 0)
+    (property "Intersheet References" "${INTERSHEET_REFS}" (id 0) (at 372.8298 71.1994 0)
       (effects (font (size 1.27 1.27)) (justify left) hide)
     )
@@
     )
   )
-  (global_label "D5_2" (shape input) (at 367.665 149.86 0) (fields_autoplaced)
+  (global_label "D5_2" (shape input) (at 27.305 67.31 180) (fields_autoplaced)
+    (effects (font (size 1.27 1.27)) (justify right))
+    (property "Intersheet References" "${INTERSHEET_REFS}" (id 0) (at 20.2352 67.2306 0)
+      (effects (font (size 1.27 1.27)) (justify right) hide)
+    )
+  )
+  (global_label "D4_2" (shape input) (at 367.665 149.86 0) (fields_autoplaced)
     (effects (font (size 1.27 1.27)) (justify left))
     (property "Intersheet References" "${INTERSHEET_REFS}" (id 0) (at 374.7348 149.7806 0)
@@
     )
   )
-  (global_label "D4_2" (shape input) (at 365.76 71.12 0) (fields_autoplaced)
-    (effects (font (size 1.27 1.27)) (justify left))
-    (property "Intersheet References" "${INTERSHEET_REFS}" (id 0) (at 372.8298 71.0406 0)
-      (effects (font (size 1.27 1.27)) (justify left) hide)
-    )
-  )
-  (global_label "D4_1" (shape input) (at 226.695 71.12 180) (fields_autoplaced)
+  (global_label "D4_1" (shape input) (at 228.6 149.86 180) (fields_autoplaced)
     (effects (font (size 1.27 1.27)) (justify right))
-    (property "Intersheet References" "${INTERSHEET_REFS}" (id 0) (at 219.6252 71.0406 0)
+    (property "Intersheet References" "${INTERSHEET_REFS}" (id 0) (at 221.5302 149.7806 0)
       (effects (font (size 1.27 1.27)) (justify right) hide)
     )
@@
     )
   )
-  (global_label "D5_1" (shape input) (at 228.6 149.86 180) (fields_autoplaced)
-    (effects (font (size 1.27 1.27)) (justify right))
-    (property "Intersheet References" "${INTERSHEET_REFS}" (id 0) (at 221.5302 149.7806 0)
-      (effects (font (size 1.27 1.27)) (justify right) hide)
+  (global_label "D5_1" (shape input) (at 166.37 67.31 0) (fields_autoplaced)
+    (effects (font (size 1.27 1.27)) (justify left))
+    (property "Intersheet References" "${INTERSHEET_REFS}" (id 0) (at 173.4398 67.2306 0)
+      (effects (font (size 1.27 1.27)) (justify left) hide)
     )
   )
@@
     )
   )
-  (global_label "D1_1" (shape input) (at 27.305 67.31 180) (fields_autoplaced)
+  (global_label "D1_1" (shape input) (at 226.695 71.12 180) (fields_autoplaced)
     (effects (font (size 1.27 1.27)) (justify right))
-    (property "Intersheet References" "${INTERSHEET_REFS}" (id 0) (at 20.2352 67.2306 0)
+    (property "Intersheet References" "${INTERSHEET_REFS}" (id 0) (at 219.6252 71.0406 0)
       (effects (font (size 1.27 1.27)) (justify right) hide)
     )
