File: irigatii2/irigatii2.kicad_pcb (KiCad board)
At the start: 2 copper layers, 11 parts, among them IC1 MIC3172YN, IC2 PCA9575PW2,118, J1 Screw_Terminal_01x02, J2 Conn_01x05, U2 OP179GRT, U3 LM4040DBZ-2.0, U4 OP179GRT

Commit message: g
Parts:
- removed J1: Screw_Terminal_01x02, TerminalBlock:TerminalBlock_Altech_AK300-2_P5.00mm
- added C1: C_Small, Capacitor_THT:CP_Axial_L11.0mm_D5.0mm_P18.00mm_Horizontal, F.Cu at (184.7, 104.3)
- added C10: 100n, Capacitor_THT:C_Disc_D3.8mm_W2.6mm_P2.50mm, F.Cu at (215.1, 103.1)
- added C13: 100n, Capacitor_THT:C_Disc_D3.8mm_W2.6mm_P2.50mm, F.Cu at (189.0, 156.0)
- added C14: 100n, Capacitor_THT:C_Disc_D3.8mm_W2.6mm_P2.50mm, F.Cu at (194.6, 156.0)
- added C15: 100n, Capacitor_THT:C_Disc_D3.8mm_W2.6mm_P2.50mm, F.Cu at (189.0, 160.2)
- added C16: 100n, Capacitor_THT:C_Disc_D3.8mm_W2.6mm_P2.50mm, F.Cu at (202.3, 143.9)
- added C17: 100n, Capacitor_THT:C_Disc_D3.8mm_W2.6mm_P2.50mm, F.Cu at (202.3, 148.0)
- added C2: C_Small, Capacitor_THT:CP_Axial_L11.0mm_D5.0mm_P18.00mm_Horizontal, F.Cu at (184.7, 97.0)
- added C3: C_Small, Capacitor_THT:CP_Axial_L11.0mm_D5.0mm_P18.00mm_Horizontal, F.Cu at (162.7, 111.6)
- added C4: C_Small, Capacitor_THT:CP_Axial_L11.0mm_D5.0mm_P18.00mm_Horizontal, F.Cu at (162.7, 104.3)
- added C5: C_Small, Capacitor_THT:CP_Axial_L11.0mm_D5.0mm_P18.00mm_Horizontal, F.Cu at (162.7, 97.0)
- added C6: C_Small, Capacitor_THT:CP_Axial_L11.0mm_D5.0mm_P18.00mm_Horizontal, F.Cu at (162.7, 119.0)
- added C7: 1u, Capacitor_THT:C_Disc_D3.8mm_W2.6mm_P2.50mm, F.Cu at (189.0, 126.0)
- added C8: 1u, Capacitor_THT:C_Disc_D3.8mm_W2.6mm_P2.50mm, F.Cu at (197.8, 117.7)
- added C9: 100n, Capacitor_THT:C_Disc_D3.8mm_W2.6mm_P2.50mm, F.Cu at (210.9, 107.3)
- added D1: D_Small, Diode_THT:D_A-405_P5.08mm_Vertical_KathodeUp, F.Cu at (189.1, 121.8)
- added D2: D_Small, Diode_THT:D_A-405_P5.08mm_Vertical_KathodeUp, F.Cu at (206.3, 103.1)
- added D3: D_Small, Diode_THT:D_A-405_P5.08mm_Vertical_KathodeUp, F.Cu at (219.6, 95.0)
- added D4: red, LED_THT:LED_D5.0mm, F.Cu at (146.7, 49.2)
- added D5: red, LED_THT:LED_D5.0mm, F.Cu at (133.4, 53.2)
- added D6: red, LED_THT:LED_D5.0mm, F.Cu at (120.1, 61.3)
- added J5: valve, TerminalBlock:TerminalBlock_Altech_AK300-2_P5.00mm, F.Cu at (164.3, 55.7)
- added J6: valve, TerminalBlock:TerminalBlock_Altech_AK300-2_P5.00mm, F.Cu at (188.8, 55.7)
- added J7: valve, TerminalBlock:TerminalBlock_Altech_AK300-2_P5.00mm, F.Cu at (176.6, 55.7)
- added J8: valve, TerminalBlock:TerminalBlock_Altech_AK300-2_P5.00mm, F.Cu at (164.3, 69.7)
- added J9: valve, TerminalBlock:TerminalBlock_Altech_AK300-2_P5.00mm, F.Cu at (164.3, 83.7)
- added Q11: PMOS, Package_TO_SOT_THT:TO-92_Wide, F.Cu at (182.9, 78.4)
- added Q12: PMOS, Package_TO_SOT_THT:TO-92_Wide, F.Cu at (207.4, 59.4)
- added Q13: PMOS, Package_TO_SOT_THT:TO-92_Wide, F.Cu at (191.1, 85.0)
- added Q14: PMOS, Package_TO_SOT_THT:TO-92_Wide, F.Cu at (199.2, 76.8)
- added Q15: NMOS, Package_TO_SOT_THT:TO-92_Inline_Wide, F.Cu at (207.4, 78.4)
- added Q16: NMOS, Package_TO_SOT_THT:TO-92_Inline_Wide, F.Cu at (199.2, 70.2)
- added Q17: NMOS, Package_TO_SOT_THT:TO-92_Inline_Wide, F.Cu at (191.1, 78.4)
- added Q18: NMOS, Package_TO_SOT_THT:TO-92_Inline_Wide, F.Cu at (223.7, 52.0)
- added Q19: NMOS, Package_TO_SOT_THT:TO-92_Inline_Wide, F.Cu at (199.2, 82.6)
- added Q20: NMOS, Package_TO_SOT_THT:TO-92_Inline_Wide, F.Cu at (182.9, 66.0)
- added Q21: NMOS, Package_TO_SOT_THT:TO-92_Inline_Wide, F.Cu at (215.5, 58.6)
- added Q22: NMOS, Package_TO_SOT_THT:TO-92_Inline_Wide, F.Cu at (223.7, 57.8)
- added Q23: PMOS, Package_TO_SOT_THT:TO-92_Wide, F.Cu at (207.4, 72.6)
- added Q24: PMOS, Package_TO_SOT_THT:TO-92_Wide, F.Cu at (191.1, 72.6)
- added Q25: PMOS, Package_TO_SOT_THT:TO-92_Wide, F.Cu at (207.4, 66.0)
- added Q26: PMOS, Package_TO_SOT_THT:TO-92_Wide, F.Cu at (199.2, 64.4)
- added Q27: NMOS, Package_TO_SOT_THT:TO-92_Inline_Wide, F.Cu at (199.2, 57.8)
- added Q28: NMOS, Package_TO_SOT_THT:TO-92_Inline_Wide, F.Cu at (174.8, 83.3)
- added Q29: NMOS, Package_TO_SOT_THT:TO-92_Inline_Wide, F.Cu at (191.1, 66.0)
- added Q30: NMOS, Package_TO_SOT_THT:TO-92_Inline_Wide, F.Cu at (182.9, 84.2)
- added Q31: NMOS, Package_TO_SOT_THT:TO-92_Inline_Wide, F.Cu at (199.2, 52.0)
- added Q32: NMOS, Package_TO_SOT_THT:TO-92_Inline_Wide, F.Cu at (215.5, 64.4)
- added Q33: NMOS, Package_TO_SOT_THT:TO-92_Inline_Wide, F.Cu at (182.9, 71.8)
- added Q34: NMOS, Package_TO_SOT_THT:TO-92_Inline_Wide, F.Cu at (174.8, 71.8)
- added Q35: PMOS, Package_TO_SOT_THT:TO-92_Wide, F.Cu at (215.5, 52.8)
- added Q36: PMOS, Package_TO_SOT_THT:TO-92_Wide, F.Cu at (207.4, 52.8)
- added Q37: NMOS, Package_TO_SOT_THT:TO-92_Inline_Wide, F.Cu at (174.8, 77.6)
- added Q38: NMOS, Package_TO_SOT_THT:TO-92_Inline_Wide, F.Cu at (174.8, 66.0)
- added R1: 100k, Resistor_THT:R_Axial_DIN0207_L6.3mm_D2.5mm_P10.16mm_Horizontal, F.Cu at (197.6, 109.6)
- added R10: 100k, Resistor_THT:R_Axial_DIN0207_L6.3mm_D2.5mm_P10.16mm_Horizontal, F.Cu at (162.3, 124.2)
- added R11: 1-10k, Resistor_THT:R_Axial_DIN0207_L6.3mm_D2.5mm_P10.16mm_Horizontal, F.Cu at (206.2, 94.9)
- added R12: 1k, Resistor_THT:R_Axial_DIN0207_L6.3mm_D2.5mm_P10.16mm_Horizontal, F.Cu at (119.2, 55.5)
- added R13: 1k, Resistor_THT:R_Axial_DIN0207_L6.3mm_D2.5mm_P10.16mm_Horizontal, F.Cu at (119.2, 51.5)
- added R16: 100k, Resistor_THT:R_Axial_DIN0207_L6.3mm_D2.5mm_P10.16mm_Horizontal, F.Cu at (184.3, 109.6)
- added R17: 1k, Resistor_THT:R_Axial_DIN0207_L6.3mm_D2.5mm_P10.16mm_Horizontal, F.Cu at (119.2, 47.4)
- added R2: 10m, Resistor_THT:R_Axial_DIN0207_L6.3mm_D2.5mm_P10.16mm_Horizontal, F.Cu at (197.6, 113.6)
- added R20: 100k, Resistor_THT:R_Axial_DIN0207_L6.3mm_D2.5mm_P10.16mm_Horizontal, F.Cu at (189.0, 147.9)
- added R21: 100k, Resistor_THT:R_Axial_DIN0207_L6.3mm_D2.5mm_P10.16mm_Horizontal, F.Cu at (162.3, 147.9)
- added R22: 100k, Resistor_THT:R_Axial_DIN0207_L6.3mm_D2.5mm_P10.16mm_Horizontal, F.Cu at (175.6, 135.7)
- added R23: 100k, Resistor_THT:R_Axial_DIN0207_L6.3mm_D2.5mm_P10.16mm_Horizontal, F.Cu at (189.0, 151.9)
- added R24: 100k, Resistor_THT:R_Axial_DIN0207_L6.3mm_D2.5mm_P10.16mm_Horizontal, F.Cu at (189.0, 143.8)
- added R25: 100k, Resistor_THT:R_Axial_DIN0207_L6.3mm_D2.5mm_P10.16mm_Horizontal, F.Cu at (162.3, 151.9)
- added R26: 100k, Resistor_THT:R_Axial_DIN0207_L6.3mm_D2.5mm_P10.16mm_Horizontal, F.Cu at (162.3, 143.8)
- added R27: 100k, Resistor_THT:R_Axial_DIN0207_L6.3mm_D2.5mm_P10.16mm_Horizontal, F.Cu at (202.3, 139.8)
- added R28: 100k, Resistor_THT:R_Axial_DIN0207_L6.3mm_D2.5mm_P10.16mm_Horizontal, F.Cu at (175.6, 139.8)
- added R29: 100k, Resistor_THT:R_Axial_DIN0207_L6.3mm_D2.5mm_P10.16mm_Horizontal, F.Cu at (175.6, 151.9)
- added R3: SOON, Resistor_THT:R_Axial_DIN0207_L6.3mm_D2.5mm_P10.16mm_Horizontal, F.Cu at (175.6, 124.2)
- added R30: 100k, Resistor_THT:R_Axial_DIN0207_L6.3mm_D2.5mm_P10.16mm_Horizontal, F.Cu at (189.0, 139.8)
- added R31: 100k, Resistor_THT:R_Axial_DIN0207_L6.3mm_D2.5mm_P10.16mm_Horizontal, F.Cu at (162.3, 156.0)
- added R32: 100k, Resistor_THT:R_Axial_DIN0207_L6.3mm_D2.5mm_P10.16mm_Horizontal, F.Cu at (175.6, 147.9)
- added R33: 100k, Resistor_THT:R_Axial_DIN0207_L6.3mm_D2.5mm_P10.16mm_Horizontal, F.Cu at (175.6, 143.8)
- added R34: 100k, Resistor_THT:R_Axial_DIN0207_L6.3mm_D2.5mm_P10.16mm_Horizontal, F.Cu at (202.3, 135.7)
- added R35: 100k, Resistor_THT:R_Axial_DIN0207_L6.3mm_D2.5mm_P10.16mm_Horizontal, F.Cu at (175.6, 156.0)
- added R36: 100k, Resistor_THT:R_Axial_DIN0207_L6.3mm_D2.5mm_P10.16mm_Horizontal, F.Cu at (189.0, 135.7)
- added R37: 100k, Resistor_THT:R_Axial_DIN0207_L6.3mm_D2.5mm_P10.16mm_Horizontal, F.Cu at (162.3, 139.8)
- added R38: 100k, Resistor_THT:R_Axial_DIN0207_L6.3mm_D2.5mm_P10.16mm_Horizontal, F.Cu at (175.6, 160.0)
- added R39: 100k, Resistor_THT:R_Axial_DIN0207_L6.3mm_D2.5mm_P10.16mm_Horizontal, F.Cu at (162.3, 160.0)
- added R4: SOON, Resistor_THT:R_Axial_DIN0207_L6.3mm_D2.5mm_P10.16mm_Horizontal, F.Cu at (184.3, 117.7)
- added R40: 100k, Resistor_THT:R_Axial_DIN0207_L6.3mm_D2.5mm_P10.16mm_Horizontal, F.Cu at (162.3, 135.7)
- added R5: 1k, Resistor_THT:R_Axial_DIN0207_L6.3mm_D2.5mm_P10.16mm_Horizontal, F.Cu at (184.3, 113.6)
- added R6: 1k, Resistor_THT:R_Axial_DIN0207_L6.3mm_D2.5mm_P10.16mm_Horizontal, F.Cu at (162.3, 128.3)
- added R7: 1k, Resistor_THT:R_Axial_DIN0207_L6.3mm_D2.5mm_P10.16mm_Horizontal, F.Cu at (206.2, 99.0)
- added R8: 100k, Resistor_THT:R_Axial_DIN0207_L6.3mm_D2.5mm_P10.16mm_Horizontal, F.Cu at (175.6, 128.3)
- added R9: 100k, Resistor_THT:R_Axial_DIN0207_L6.3mm_D2.5mm_P10.16mm_Horizontal, F.Cu at (132.5, 47.4)
- JP2: value Adress0 -> Adress1
- JP3: value Adress0 -> Adress2
- JP4: value Adress0 -> Adress3
Connections:
- IC1 pad 4: unconnected-(IC1-Pad4) -> EN
- IC2 pad 10: unconnected-(IC2-Pad10) -> D3_1
- IC2 pad 11: unconnected-(IC2-Pad11) -> D3_2
- IC2 pad 12: unconnected-(IC2-Pad12) -> D3_3
- IC2 pad 13: unconnected-(IC2-Pad13) -> D3_4
- IC2 pad 17: unconnected-(IC2-Pad17) -> D5_2
- IC2 pad 18: unconnected-(IC2-Pad18) -> D5_1
- IC2 pad 19: unconnected-(IC2-Pad19) -> D4_2
- IC2 pad 20: unconnected-(IC2-Pad20) -> D4_1
- IC2 pad 23: unconnected-(IC2-Pad23) -> LED_3
- IC2 pad 24: unconnected-(IC2-Pad24) -> LED_2
- IC2 pad 25: unconnected-(IC2-Pad25) -> LED_1
- IC2 pad 26: unconnected-(IC2-Pad26) -> EN
- IC2 pad 4: unconnected-(IC2-Pad4) -> D1_1
- IC2 pad 5: unconnected-(IC2-Pad5) -> D1_2
- IC2 pad 6: unconnected-(IC2-Pad6) -> D2_1
- IC2 pad 7: unconnected-(IC2-Pad7) -> D2_2

Commit message: h
Parts:
- added RV1: R_Potentiometer, Potentiometer_THT:Potentiometer_ACP_CA9-V10_Vertical, F.Cu at (82.7, 85.0)
- moved C10 191.0 mm to (37.9, 174.4), turned to -90 degrees
- moved C9 179.4 mm to (44.5, 174.5), turned to -90 degrees
- moved C8 160.8 mm to (41.7, 156.5), turned to 90 degrees
- moved IC2 105.4 mm to (41.5, 164.2), turned to 90 degrees
- moved J2 87.2 mm to (31.4, 158.1)
Connections:
- J2 pad 2: I2C_CLK -> I2C_SDA
- J2 pad 3: I2C_SDA -> I2C_CLK
- R11 pad 1: Net-(R11-Pad1) -> +3V3
- R2 pad 1: Net-(R11-Pad1) -> +3V3
- R5 pad 1: Net-(R11-Pad1) -> +3V3
Routing:
- added copper zone on B.Cu, net GND

Commit message: j
Parts:
- R20, R21, R22, R23, R24, R25, R26, R27, R28, R29, R30, R31, R32, R33, R35, R36, R37, R38, R39, R40: footprint Resistor_THT:R_Axial_DIN0207_L6.3mm_D2.5mm_P10.16mm_Horizontal -> Resistor_THT:R_Axial_DIN0204_L3.6mm_D1.6mm_P5.08mm_Vertical
- R34: footprint Resistor_THT:R_Axial_DIN0207_L6.3mm_D2.5mm_P10.16mm_Horizontal -> Resistor_THT:R_Axial_DIN0204_L3.6mm_D1.6mm_P5.08mm_Horizontal
- moved Q35 191.0 mm to (63.0, 167.7)
- moved Q21 166.8 mm to (97.1, 176.0)
- moved Q36 163.8 mm to (88.3, 165.3), turned to 180 degrees
- moved Q22 155.4 mm to (122.3, 175.6), turned to 180 degrees
- moved Q18 154.5 mm to (122.4, 168.6), turned to 180 degrees
- moved Q37 147.7 mm to (63.0, 174.2)
- moved J6 143.5 mm to (106.9, 173.5)
- moved R27 141.4 mm to (69.8, 90.3), turned to 90 degrees
- moved Q12 140.6 mm to (73.3, 101.5)
- moved Q38 137.4 mm to (88.1, 172.6), turned to 180 degrees
- moved Q17 130.1 mm to (97.1, 168.4)
- moved Q16 128.1 mm to (73.4, 93.9)
- moved Q23 125.6 mm to (110.7, 152.8), turned to 90 degrees
- moved J9 125.5 mm to (73.0, 169.7)
- moved Q31 125.2 mm to (124.8, 152.6), turned to 90 degrees
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Other:
- board outline added: 100 x 100 mm

Commit message: g
Parts:
- removed U3: LM4040DBZ-2.0, Package_TO_SOT_SMD:SOT-23
- removed U4: OP179GRT, Package_TO_SOT_SMD:SOT-23-5
- added C11: 1u, Capacitor_THT:C_Disc_D3.8mm_W2.6mm_P2.50mm, F.Cu at (52.7, 104.3)
- added C12: 1u, Capacitor_THT:C_Disc_D3.8mm_W2.6mm_P2.50mm, F.Cu at (63.1, 109.7)
- added T1: Transformer_1P_1S, Coils:TRANSFORMER, F.Cu at (40.7, 145.4)
- added U1: NJM2114, Package_DIP:DIP-8_W7.62mm_LongPads, F.Cu at (45.0, 109.9)
- C10, C8, C9: footprint Capacitor_THT:C_Disc_D3.8mm_W2.6mm_P2.50mm -> Capacitor_SMD:C_0805_2012Metric_Pad1.18x1.45mm_HandSolder
- C2: footprint Capacitor_THT:CP_Axial_L11.0mm_D5.0mm_P18.00mm_Horizontal -> Capacitor_THT:C_Disc_D4.3mm_W1.9mm_P5.00mm
- D2: footprint Diode_THT:D_A-405_P5.08mm_Vertical_KathodeUp -> Diode_THT:D_A-405_P10.16mm_Horizontal
- R1, R10, R12, R13, R16, R17, R5, R6, R7, R8, R9: footprint Resistor_THT:R_Axial_DIN0207_L6.3mm_D2.5mm_P10.16mm_Horizontal -> Resistor_THT:R_Axial_DIN0204_L3.6mm_D1.6mm_P5.08mm_Vertical
- R11: value 1-10k -> 120; footprint Resistor_THT:R_Axial_DIN0207_L6.3mm_D2.5mm_P10.16mm_Horizontal -> Resistor_THT:R_Axial_DIN0204_L3.6mm_D1.6mm_P5.08mm_Vertical
- U2: value OP179GRT -> TL431LP; footprint Package_TO_SOT_SMD:SOT-23-5 -> Package_TO_SOT_THT:TO-92_Inline
- moved C1 219.8 mm to (-34.5, 121.7), turned to 90 degrees
- moved C5 209.8 mm to (-41.8, 143.6), turned to 90 degrees
- moved C4 201.1 mm to (-34.5, 143.6), turned to 90 degrees
- moved C3 192.6 mm to (-27.1, 143.6), turned to 90 degrees
- moved D3 190.0 mm to (33.5, 133.3), turned to 90 degrees
- moved C6 184.2 mm to (-19.8, 143.6), turned to 90 degrees
- moved D2 168.7 mm to (46.0, 155.4), turned to 180 degrees
- moved R1 167.8 mm to (31.8, 135.9)
- moved R16 165.6 mm to (18.8, 102.1), turned to 90 degrees
- moved R2 164.9 mm to (32.8, 108.7), turned to -90 degrees
- moved IC1 163.2 mm to (41.2, 128.7), turned to -90 degrees
- moved R7 158.5 mm to (51.6, 134.0), turned to 90 degrees
- moved JP2 158.4 mm to (42.6, 105.1)
- moved JP1 158.1 mm to (36.6, 100.7), turned to 90 degrees
- moved C2 158.1 mm to (29.6, 127.9), turned to -90 degrees
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Connections:
- U2 pad 1: Net-(R10-Pad1) -> /2V
- U2 pad 2: unconnected-(U2-Pad2) -> GND
- U2 pad 3: Net-(R10-Pad2) -> /2V
Routing:
- net +12V: track 0.00 -> 235.0 mm
- net +3V3: track 0.00 -> 86.8 mm
- net Net-(C2-Pad1): track 0.00 -> 35.0 mm
- net Net-(C16-Pad1): track 0.00 -> 33.3 mm
- net Net-(C15-Pad1): track 0.00 -> 33.1 mm
- net Net-(C13-Pad1): track 0.00 -> 32.5 mm
- net Net-(J7-Pad1): track 0.00 -> 32.4 mm
- net Net-(C14-Pad1): track 0.00 -> 32.1 mm
- net Net-(J8-Pad1): track 0.00 -> 31.6 mm
- net Net-(J9-Pad1): track 0.00 -> 30.8 mm
- net Net-(C17-Pad1): track 0.00 -> 30.6 mm
- net Net-(J6-Pad1): track 0.00 -> 30.5 mm
- net Net-(Q23-Pad2): track 0.00 -> 25.2 mm
- net IC_FBpin: track 0.00 -> 23.5 mm
- net Net-(Q11-Pad2): track 0.00 -> 22.7 mm
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
Commit message: d
Parts:
- added C18: 22u, Capacitor_THT:CP_Radial_D5.0mm_P2.00mm, F.Cu at (53.3, 155.6)
- added C19: 22u, Capacitor_THT:CP_Radial_D5.0mm_P2.00mm, F.Cu at (53.5, 163.5)
- added C20: 220u, Capacitor_THT:CP_Radial_D8.0mm_P3.80mm, F.Cu at (83.6, 154.9)
- added C21: 220u, Capacitor_THT:CP_Radial_D8.0mm_P3.80mm, F.Cu at (100.3, 106.8)
- added C22: 220u, Capacitor_THT:CP_Radial_D8.0mm_P3.80mm, F.Cu at (103.1, 139.6)
- C1, C3, C4, C6: value C_Small -> 220u; footprint Capacitor_THT:CP_Axial_L11.0mm_D5.0mm_P18.00mm_Horizontal -> Capacitor_THT:CP_Radial_D8.0mm_P3.80mm
- C5: value C_Small -> 1u; footprint Capacitor_THT:CP_Axial_L11.0mm_D5.0mm_P18.00mm_Horizontal -> Capacitor_THT:C_Disc_D4.3mm_W1.9mm_P5.00mm
- moved C4 132.6 mm to (97.7, 155.2)
- moved C3 131.7 mm to (103.3, 125.5), turned to 180 degrees
- moved C1 107.9 mm to (68.1, 155.3)
- moved C6 105.3 mm to (78.9, 106.8), turned to -90 degrees
- moved C5 87.1 mm to (44.9, 135.4), turned to 180 degrees
- moved R16 23.7 mm to (29.7, 123.1), turned to 0 degrees
- moved U2 3.70 mm to (62.6, 110.9)
- moved C12 3.35 mm to (66.3, 110.7)
- moved R11 1.24 mm to (56.4, 105.4)
- moved R9 0.67 mm to (49.3, 101.9)
Connections:
- C5 pad 1: +12V -> GND
- C5 pad 2: GND -> Net-(C2-Pad1)
- C6 pad 1: GND -> +12V
- C6 pad 2: Net-(C2-Pad1) -> GND
- IC2 pad 10: D3_1 -> D2_2
- IC2 pad 11: D3_2 -> D2_1
- IC2 pad 12: D3_3 -> D1_1
- IC2 pad 13: D3_4 -> D1_2
- IC2 pad 4: D1_1 -> D3_1
- IC2 pad 5: D1_2 -> D3_2
- IC2 pad 6: D2_1 -> D3_3
- IC2 pad 7: D2_2 -> D3_4
- Q19 pad 1: D1_1 -> D5_2
- Q20 pad 1: D1_2 -> D5_1
- Q21 pad 1: D4_1 -> D1_1
- Q22 pad 1: D4_2 -> D1_2
- Q33 pad 1: D5_1 -> D4_1
- Q34 pad 1: D5_2 -> D4_2
- R26 pad 2: D1_1 -> D5_2
- R27 pad 2: D1_2 -> D5_1
- R28 pad 2: D4_1 -> D1_1
- R29 pad 2: D4_2 -> D1_2
- R38 pad 2: D5_1 -> D4_1
- R39 pad 2: D5_2 -> D4_2
Routing:
- net D1_2: track 4.05 -> 134.4 mm, vias 0 -> 7
- net D2_1: track 3.41 -> 129.1 mm, vias 0 -> 6
- net D1_1: track 3.24 -> 112.1 mm, vias 0 -> 6
- net D3_4: track 0.00 -> 108.5 mm, vias 0 -> 6
- net D3_3: track 0.00 -> 103.1 mm, vias 0 -> 6
- net D3_2: track 0.00 -> 100.4 mm, vias 0 -> 6
- net D4_1: track 3.37 -> 103.5 mm, vias 0 -> 6
- net D4_2: track 3.54 -> 102.0 mm, vias 0 -> 6
- net +12V: track 235.0 -> 331.4 mm
- net D3_1: track 0.00 -> 94.1 mm, vias 0 -> 8
- net D2_2: track 3.34 -> 95.7 mm, vias 0 -> 6
- net D5_2: track 3.56 -> 69.7 mm
- net EN: track 0.00 -> 38.1 mm, vias 0 -> 6
- net D5_1: track 3.74 -> 38.0 mm
- net Net-(IC2-Pad3): track 0.00 -> 12.4 mm, vias 0 -> 2
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
Commit message: v
Parts:
- added C23: 500+u, Capacitor_THT:CP_Radial_D13.0mm_P5.00mm, F.Cu at (102.1, 121.8)
- added H1: MountingHole_Pad, MountingHole:MountingHole_3.2mm_M3_Pad_TopBottom, F.Cu at (32.0, 86.0)
- added H2: MountingHole_Pad, MountingHole:MountingHole_3.2mm_M3_Pad_TopBottom, F.Cu at (122.0, 86.0)
- added H3: MountingHole_Pad, MountingHole:MountingHole_3.2mm_M3_Pad_TopBottom, F.Cu at (122.0, 176.0)
- added H4: MountingHole_Pad, MountingHole:MountingHole_3.2mm_M3_Pad_TopBottom, F.Cu at (32.0, 176.0)
- added H5: MountingHole_Pad, MountingHole:MountingHole_3.2mm_M3_Pad_TopBottom, F.Cu at (81.5, 130.9)
- added kibuzzard-633BE47A: G***, kibuzzard-633BE47A, F.Cu at (40.4, 169.8)
- added kibuzzard-633BE88B: G***, kibuzzard-633BE88B, F.Cu at (30.7, 164.7)
- C1, C20, C21, C22, C3, C4, C6: value 220u -> 500+u; footprint Capacitor_THT:CP_Radial_D8.0mm_P3.80mm -> Capacitor_THT:CP_Radial_D13.0mm_P5.00mm
- moved C21 51.0 mm to (81.7, 154.3), turned to 90 degrees
- moved C3 47.8 mm to (62.7, 150.7), turned to 0 degrees
- moved C1 36.4 mm to (74.1, 119.4), turned to 0 degrees
- moved C22 34.1 mm to (89.4, 108.3), turned to -90 degrees
- moved C6 30.3 mm to (68.5, 135.3), turned to 0 degrees
- moved C4 19.1 mm to (101.7, 136.6), turned to 180 degrees
- moved C20 17.8 mm to (101.2, 152.7), turned to 180 degrees
- moved C17 17.4 mm to (63.7, 165.4), turned to 90 degrees
- moved J9 15.4 mm to (58.1, 173.5)
- moved Q38 15.3 mm to (73.1, 175.4)
- moved Q37 15.2 mm to (48.0, 176.1)
- moved Q36 15.1 mm to (73.4, 167.7)
- moved R40 14.9 mm to (60.7, 160.4), turned to -90 degrees
- moved Q35 13.2 mm to (49.8, 166.4), turned to -90 degrees
- moved Q26 12.4 mm to (108.2, 99.4), turned to 90 degrees
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Connections:
- R6 pad 1: Net-(R10-Pad2) -> Net-(C2-Pad1)
- R6 pad 2: Net-(C2-Pad1) -> Net-(R10-Pad2)
Routing:
- net Net-(Q26-Pad2): track 18.0 -> 31.7 mm
- net Net-(J8-Pad1): track 31.6 -> 19.9 mm
- net D1_1: track 112.1 -> 123.0 mm
- net D1_2: track 134.4 -> 126.6 mm, vias 7 -> 5
- net Net-(J9-Pad1): track 30.8 -> 23.2 mm
- net Net-(C17-Pad1): track 30.6 -> 23.3 mm
- net D3_2: track 100.4 -> 105.3 mm
- net D3_1: track 94.1 -> 98.5 mm, vias 8 -> 6
- net D3_3: track 103.1 -> 106.8 mm
- net I2C_SDA: track 9.06 -> 11.3 mm
- net D2_1: track 129.1 -> 131.0 mm
- net +3V3: track 83.4 -> 81.5 mm
- net Net-(Q24-Pad2): track 18.6 -> 16.8 mm
- net Net-(C17-Pad2): track 2.53 -> 4.13 mm
- net GND: track 22.3 -> 23.8 mm, vias 13 -> 15
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Other:
- outline, holes or cut-outs redrawn
