File: irigatii2/irigatii2.kicad_sch (KiCad schematic)
At the start: 55 parts, among them IC1 MIC3172YN, IC2 PCA9575PW2,118, J2 Conn_01x05, T1 Transformer_1P_1S, U1 NJM2114, U2 TL431LP

Commit message: g
Parts:
- added J1: Conn_01x02, Connector_PinHeader_2.54mm:PinHeader_1x02_P2.54mm_Vertical, symbol Connector_Generic:Conn_01x02
- added JP5: Jumper_2_Open, Jumper:SolderJumper-2_P1.3mm_Open_Pad1.0x1.5mm, symbol Jumper:Jumper_2_Open
Connections:
- net +3V3: now also JP5.2 (B)
- net +5V: now also J1.1 (Pin_1), J1.2 (Pin_2), JP5.1 (A)
Changed lines of the file:
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@@
   (junction (at 294.005 139.065) (diameter 0) (color 0 0 0 0)
   )
+  (junction (at 356.87 117.475) (diameter 0) (color 0 0 0 0)
+  )
+  (junction (at 356.87 120.015) (diameter 0) (color 0 0 0 0)
+  )
   (junction (at 184.15 60.96) (diameter 0) (color 0 0 0 0)
   )
@@
     (stroke (width 0) (type default) (color 0 0 0 0))
   )
+  (wire (pts (xy 356.87 114.935) (xy 356.87 117.475))
+    (stroke (width 0) (type default) (color 0 0 0 0))
+  )
   (wire (pts (xy 184.15 25.4) (xy 227.33 25.4))
     (stroke (width 0) (type default) (color 0 0 0 0))
@@
     (stroke (width 0) (type default) (color 0 0 0 0))
   )
+  (wire (pts (xy 356.87 117.475) (xy 351.155 117.475))
+    (stroke (width 0) (type default) (color 0 0 0 0))
+  )
   (wire (pts (xy 294.005 128.905) (xy 294.005 133.985))
     (stroke (width 0) (type default) (color 0 0 0 0))
@@
     (stroke (width 0) (type default) (color 0 0 0 0))
   )
+  (wire (pts (xy 374.65 120.015) (xy 379.095 120.015))
+    (stroke (width 0) (type default) (color 0 0 0 0))
+  )
   (wire (pts (xy 325.12 71.755) (xy 325.12 84.455))
     (stroke (width 0) (type default) (color 0 0 0 0))
@@
     (stroke (width 0) (type default) (color 0 0 0 0))
   )
+  (wire (pts (xy 356.87 117.475) (xy 356.87 120.015))
+    (stroke (width 0) (type default) (color 0 0 0 0))
+  )
   (wire (pts (xy 184.15 60.96) (xy 196.85 60.96))
     (stroke (width 0) (type default) (color 0 0 0 0))
@@
     (stroke (width 0) (type default) (color 0 0 0 0))
   )
+  (wire (pts (xy 356.87 120.015) (xy 364.49 120.015))
+    (stroke (width 0) (type default) (color 0 0 0 0))
+  )
   (wire (pts (xy 99.06 123.19) (xy 101.6 123.19))
     (stroke (width 0) (type default) (color 0 0 0 0))
@@
     (stroke (width 0) (type default) (color 0 0 0 0))
   )
+  (wire (pts (xy 351.155 120.015) (xy 356.87 120.015))
+    (stroke (width 0) (type default) (color 0 0 0 0))
+  )
   (wire (pts (xy 236.22 129.54) (xy 236.22 131.445))
     (stroke (width 0) (type default) (color 0 0 0 0))
@@
     )
   )
+  (global_label "current_in" (shape input) (at 92.71 27.94 180) (fields_autoplaced)
+    (effects (font (size 1 1)) (justify right))
+    (property "Intersheet References" "${INTERSHEET_REFS}" (id 0) (at 83.3338 27.8775 0)
+      (effects (font (size 1 1)) (justify right) hide)
+    )
+  )
   (global_label "D1_1" (shape input) (at 55.88 140.97 180) (fields_autoplaced)
     (effects (font (size 1.27 1.27)) (justify right))
@@
     )
   )
+  (global_label "current_in" (shape input) (at 379.095 120.015 0) (fields_autoplaced)
+    (effects (font (size 1 1)) (justify left))
+    (property "Intersheet References" "${INTERSHEET_REFS}" (id 0) (at 388.4712 120.0775 0)
+      (effects (font (size 1 1)) (justify left) hide)
+    )
+  )
   (global_label "D5_2" (shape input) (at 101.6 140.97 0) (fields_autoplaced)
     (effects (font (size 1.27 1.27)) (justify left))
@@
     (pin "1")
   )
+  (symbol (lib_id "Connector_Generic:Conn_01x02") (at 346.075 120.015 180) (unit 1)
+    (in_bom no) (on_board yes) (fields_autoplaced)
+    (property "Reference" "J1" (id 0) (at 346.075 110.49 0))
+    (property "Value" "Conn_01x02" (id 1) (at 346.075 113.03 0))
+    (property "Footprint" "Connector_PinHeader_2.54mm:PinHeader_1x02_P2.54mm_Vertical" (id 2) (at 346.075 120.015 0)
+      (effects (font (size 1.27 1.27)) hide)
+    )
+    (property "Datasheet" "~" (id 3) (at 346.075 120.015 0)
+      (effects (font (size 1.27 1.27)) hide)
+    )
+    (pin "1")
+    (pin "2")
+  )
   (symbol (lib_id "power:GND") (at 176.53 140.97 0) (unit 1)
     (in_bom yes) (on_board yes) (fields_autoplaced)
@@
     (pin "1")
   )
+  (symbol (lib_id "Jumper:Jumper_2_Open") (at 369.57 120.015 0) (unit 1)
+    (in_bom no) (on_board yes) (fields_autoplaced)
+    (property "Reference" "JP5" (id 0) (at 369.57 113.03 0))
+    (property "Value" "Jumper_2_Open" (id 1) (at 369.57 115.57 0))
+    (property "Footprint" "Jumper:SolderJumper-2_P1.3mm_Open_Pad1.0x1.5mm" (id 2) (at 369.57 120.015 0)
+      (effects (font (size 1.27 1.27)) hide)
+    )
+    (property "Datasheet" "~" (id 3) (at 369.57 120.015 0)
+      (effects (font (size 1.27 1.27)) hide)
+    )
+    (pin "1")
+    (pin "2")
+  )
   (symbol (lib_id "Device:D_Small") (at 138.43 69.85 180) (unit 1)
     (in_bom yes) (on_board yes) (fields_autoplaced)
@@
     (pin "1")
   )
+  (symbol (lib_id "power:+5V") (at 356.87 114.935 0) (unit 1)
+    (in_bom yes) (on_board yes) (fields_autoplaced)
+    (property "Reference" "#PWR0140" (id 0) (at 356.87 118.745 0)
+      (effects (font (size 1.27 1.27)) hide)
+    )
+    (property "Value" "+5V" (id 1) (at 356.87 109.855 0))
+    (property "Footprint" "" (id 2) (at 356.87 114.935 0)
+      (effects (font (size 1.27 1.27)) hide)
+    )
+    (property "Datasheet" "" (id 3) (at 356.87 114.935 0)
+      (effects (font (size 1.27 1.27)) hide)
+    )
+    (pin "1")
+  )
   (symbol (lib_id "power:GND") (at 139.7 140.97 0) (unit 1)
     (in_bom yes) (on_board yes) (fields_autoplaced)
@@
       (reference "#PWR0139") (unit 1) (value "+12V") (footprint "")
     )
+    (path "/c91d3fbb-b181-48f6-9726-6677175d4e75"
+      (reference "#PWR0140") (unit 1) (value "+5V") (footprint "")
+    )
     (path "/15ac21d5-9c0d-4dcf-b906-d2a3e2e6e333"
       (reference "#PWR0142") (unit 1) (value "+12V") (footprint "")
@@
       (reference "IC2") (unit 1) (value "PCA9575PW2,118") (footprint "SamacSys_Parts:SOP65P640X110-28N")
     )
+    (path "/a59f2534-f80b-466e-8b0c-91c36212e800"
+      (reference "J1") (unit 1) (value "Conn_01x02") (footprint "Connector_PinHeader_2.54mm:PinHeader_1x02_P2.54mm_Vertical")
+    )
     (path "/61c4b3e7-390f-4204-9128-24ba46c82c08"
       (reference "J2") (unit 1) (value "Conn_01x05") (footprint "Connector_PinHeader_2.54mm:PinHeader_1x05_P2.54mm_Vertical")
@@
       (reference "JP4") (unit 1) (value "Adress3") (footprint "Jumper:SolderJumper-3_P1.3mm_Bridged12_Pad1.0x1.5mm")
     )
+    (path "/b8305017-eeb9-4b25-87d8-5541ecb8aa1b"
+      (reference "JP5") (unit 1) (value "Jumper_2_Open") (footprint "Jumper:SolderJumper-2_P1.3mm_Open_Pad1.0x1.5mm")
+    )
     (path "/ab4119c1-34ff-423b-afbe-884f69617533/6112b8e6-1705-4833-9140-a4b062282a5c"
